File: CPU-RK3399_PWM.kicad_sch (KiCad schematic)
At the start: 1 part, among them U1 RK3399

Commit message: design PMIC
Parts:
- removed U1: RK3399, footprints:BGA828C65P31X31_2100X2100X161, symbol component_library:System On Chip (SoC)/RK3399
Connections:
- no-connect marks 1 -> 0
