File: Camera.kicad_sch (KiCad schematic)
At the start: 0 parts

Commit message: design CPU-RK3399 eMMC Controller
Other:
- company: (none) -> TickLab
Changed lines of the file:
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@@
 	(paper "A4")
 	(title_block
-		(date "2026-01-09")
+		(date "2026-01-14")
 		(rev "1.0.0")
+		(company "TickLab")
 	)
 	(bus_alias "CAM_CSI1_D"
