File: RJ45.kicad_sch (KiCad schematic)
At the start: 0 parts

Commit message: create netclass
Changed lines of the file:
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@@
 		)
 	)
-	(label "MDI0+"
+	(label "PHY_MDI0+"
 		(at 134.62 86.36 0)
 		(effects
@@
 		)
 	)
-	(label "MDI0-"
+	(label "PHY_MDI0-"
 		(at 134.62 88.9 0)
 		(effects
@@
 		)
 	)
-	(label "MDI1-"
+	(label "PHY_MDI1-"
 		(at 134.62 93.98 0)
 		(effects
@@
 		)
 	)
-	(label "MDI1+"
+	(label "PHY_MDI1+"
 		(at 134.62 91.44 0)
 		(effects

Commit message: design CPU-RK3399 eMMC Controller
Other:
- company: (none) -> TickLab
Changed lines of the file:
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@@
 	(paper "A4")
 	(title_block
-		(date "2026-01-09")
+		(date "2026-01-14")
 		(rev "1.0.0")
+		(company "TickLab")
 	)
 	(wire
