File: microSD.kicad_sch (KiCad schematic)
At the start: 0 parts

Commit message: update root schematic
Changed lines of the file:
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@@
 		(rev "1.0.0")
+	)
+	(wire
+		(pts
+			(xy 88.9 144.78) (xy 106.68 144.78)
+		)
+		(stroke
+			(width 0)
+			(type default)
+		)
+	)
+	(wire
+		(pts
+			(xy 88.9 149.86) (xy 106.68 149.86)
+		)
+		(stroke
+			(width 0)
+			(type default)
+		)
+	)
+	(wire
+		(pts
+			(xy 88.9 142.24) (xy 106.68 142.24)
+		)
+		(stroke
+			(width 0)
+			(type default)
+		)
+	)
+	(bus
+		(pts
+			(xy 88.9 147.32) (xy 106.68 147.32)
+		)
+		(stroke
+			(width 0)
+			(type default)
+		)
 	)
 	(label "MSD_CLX"
@@
 	)
 	(hierarchical_label "CMD"
-		(shape output)
+		(shape bidirectional)
 		(at 88.9 144.78 180)
 		(effects

Commit message: design CPU-RK3399 eMMC Controller
Other:
- company: (none) -> TickLab
Changed lines of the file:
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@@
 	(paper "A4")
 	(title_block
-		(date "2026-01-09")
+		(date "2026-01-14")
 		(rev "1.0.0")
+		(company "TickLab")
 	)
 	(wire
