File: Power_DC-IN.kicad_sch (KiCad schematic)
At the start: 65 parts, among them U5 TPS25974ARPWR, U6 TPS548A28RWWR, U7 TPS51386RJNR

Commit message: update design power
Parts:
- renumbered C152 to C164, C153 to C165, C154 to C166, C155 to C167, C156 to C168, C157 to C169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
