File: Power_PMIC.kicad_sch (KiCad schematic)
At the start: 78 parts, among them U2 RK808-D

Commit message: update design power
Parts:
- removed L1, L2, L5, L6: ~, footprints:ETQP3M1R5KVP, symbol component_library:Inductors/ETQP3M1R5KVP
- removed R67: ~, footprints:RESC1608X45N, symbol component_library:Resistors/0603WAF0000T5E
- removed R68: ~, footprints:RESC1005X35N, symbol component_library:Resistors/0402WGF2003TCE
- removed R69: ~, footprints:RESC1005X35N, symbol component_library:Resistors/0402WGF5102TCE
- added L3: ~, footprints:CRH201610S-1R0MT, symbol component_library:Inductors/CRH201610S-1R0MT
- added L4: ~, footprints:VLS201610CX-2R2M-1, symbol component_library:Inductors/VLS201610CX-2R2M-1
- added L5: ~, footprints:FXLB252012-2R2-M, symbol component_library:Inductors/FXLB252012-2R2-M
- added L6: ~, footprints:NRSE2512-1R0M, symbol component_library:Inductors/NRSE2512-1R0M
- added R90: ~, footprints:RESC1608X45N, symbol component_library:Resistors/0603WAF1203T5E
- added R92: ~, footprints:RESC1005X35N, symbol component_library:Resistors/0402WGF4302TCE
- renumbered BTN3 to BTN2, BTN2 to BTN3, C118 to C152, C126 to C153, C120 to C154, C119 to C155, C121 to C156, C128 to C157, C127 to C158, C129 to C159, C122 to C160, C130 to C161, C133 to C162, C131 to C163, C132 to C164, C123 to C165, C124 to C166, C125 to C167, C134 to C168, C145 to C169, C137 to C170, C135 to C171, C138 to C172, C139 to C173, C136 to C174, C140 to C175, C146 to C176, C141 to C177, C147 to C178, C143 to C179, C148 to C180, C144 to C181, C149 to C182, C142 to C183, C150 to C184, C186 to C185, C151 to C186, C189 to C187, C197 to C188, C187 to C189, C188 to C192, C192 to C193, C193 to C194, C196 to C195, C194 to C196, C195 to C197, D2 to D4, D9 to D5, D3 to D6, D6 to D9, R78 to R100, R77 to R101, R65 to R88, R70 to R89, R66 to R91, R79 to R93, R72 to R94, R71 to R95, R75 to R96, R73 to R97, R74 to R98, R76 to R99, U2 to U5
Connections:
- net +0V9_VDD_CENTER: now also L3.1
- net +0V9_VDD_CPU_L: now also L6.1
- net +1V35_VCC_DDR: now also L5.2
- net +1V8_VCC: now also L4.2
- net 0V9_VDD_CENTER_SW: now also L3.2
- net 0V9_VDD_CPU_L_SW: now also L6.2
- net 1V35_VCC_DDR_FB: now also R90.1, R92.1
- net 1V35_VCC_DDR_SW: now also L5.1
- net 1V8_VCC_SW: now also L4.1
- net GND: now also R90.2
- net at R89.2: now also R92.2
Other:
- note added: "DDR3: 1.5V DDR3L: 1.35V LPDDR3: 1.25V LPDDR4: 1.13V"
- note added: "Trace > 1.5A"
- note added: "Trace > 1A"
- note added: "Trace > 2A"
- note added: "Trace > 3A"
