File: CPU-RK3399.kicad_sch (KiCad schematic)
At the start: 0 parts

Commit message: design PMIC
Other:
- sheet CPU-RK3399 UART renamed CPU-RK3399 Protocols
- removed sheet CPU-RK3399 I2C
- removed sheet CPU-RK3399 I2S
- removed sheet CPU-RK3399 ISP
- removed sheet CPU-RK3399 PWM
- removed sheet CPU-RK3399 SPI
- added sheet CPU-RK3399 PCIe (CPU-RK3399_PCIe.kicad_sch)
- sheet CPU-RK3399 PMU Controller ports: added GPIO1_C7, GPIO1_D0; removed none
- sheet CPU-RK3399 Protocols: file CPU-RK3399_UART.kicad_sch -> CPU-RK3399_Protocols.kicad_sch
- sheet CPU-RK3399 Protocols ports: added I2C0; removed none

Commit message: update design power
Other:
- sheet CPU-RK3399 Protocols ports: added GPIO1_B6, GPIO1_C1; removed none
Changed lines of the file:
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@@
+	(wire
+		(pts
+			(xy 142.24 30.48) (xy 144.78 30.48)
+		)
+		(stroke
+			(width 0)
+			(type default)
+		)
+	)
 	(wire
 		(pts
@@
 		(pts
 			(xy 45.72 40.64) (xy 48.26 40.64)
+		)
+		(stroke
+			(width 0)
+			(type default)
+		)
+	)
+	(wire
+		(pts
+			(xy 142.24 27.94) (xy 144.78 27.94)
 		)
 		(stroke
@@
 		)
 	)
+	(hierarchical_label "GPIO1_C1"
+		(shape output)
+		(at 144.78 27.94 0)
+		(effects
+			(font
+				(size 1.27 1.27)
+			)
+			(justify left)
+		)
+	)
 	(hierarchical_label "WLBT_GPIO"
 		(shape bidirectional)
@@
 			)
 			(justify right)
+		)
+	)
+	(hierarchical_label "GPIO1_B6"
+		(shape output)
+		(at 144.78 30.48 0)
+		(effects
+			(font
+				(size 1.27 1.27)
+			)
+			(justify left)
 		)
 	)
@@
 			(effects
 				(font
+					(size 1.27 1.27)
+				)
+				(justify right)
+			)
+		)
+		(pin "GPIO1_C1" output
+			(at 142.24 27.94 0)
+			(effects
+				(font
+					(size 1.27 1.27)
+				)
+				(justify right)
+			)
+		)
+		(pin "GPIO1_B6" output
+			(at 142.24 30.48 0)
+			(effects
+				(font

Commit message: finish design power
Other:
- sheet CPU-RK3399 Protocols ports: added PWM2; removed none
Changed lines of the file:
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@@
+	(wire
+		(pts
+			(xy 142.24 33.02) (xy 144.78 33.02)
+		)
+		(stroke
+			(width 0)
+			(type default)
+		)
+	)
 	(wire
 		(pts
@@
 		(shape output)
 		(at 83.82 40.64 0)
+		(effects
+			(font
+				(size 1.27 1.27)
+			)
+			(justify left)
+		)
+	)
+	(hierarchical_label "PWM2"
+		(shape output)
+		(at 144.78 33.02 0)
 		(effects
 			(font
@@
 			(effects
 				(font
+					(size 1.27 1.27)
+				)
+				(justify right)
+			)
+		)
+		(pin "PWM2" output
+			(at 142.24 33.02 0)
+			(effects
+				(font

Commit message: design DDR
Other:
- sheet CPU-RK3399 PMU Controller ports: added GPIO4_D2; removed none
- sheet CPU-RK3399 Protocols ports: added GPIO1_A1, GPIO1_A2, GPIO1_A3; removed none
- sheet CPU-RK3399 USB ports: added TYPEC0_U2VBUSDET, TYPEC1_U2VBUSDET; removed none
Changed lines of the file:
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@@
 	(wire
 		(pts
+			(xy 228.6 83.82) (xy 231.14 83.82)
+		)
+		(stroke
+			(width 0)
+			(type default)
+		)
+	)
+	(wire
+		(pts
 			(xy 190.5 111.76) (xy 210.82 111.76)
 		)
@@
 		)
 	)
-	(wire
-		(pts
-			(xy 7.62 106.68) (xy 30.48 106.68)
-		)
-		(stroke
-			(width 0)
-			(type default)
-		)
-	)
 	(bus
 		(pts
@@
 	(bus
 		(pts
-			(xy 68.58 106.68) (xy 71.12 106.68)
+			(xy 68.58 109.22) (xy 71.12 109.22)
 		)
 		(stroke
@@
 	(wire
 		(pts
+			(xy 68.58 116.84) (xy 71.12 116.84)
+		)
+		(stroke
+			(width 0)
+			(type default)
+		)
+	)
+	(wire
+		(pts
 			(xy 208.28 50.8) (xy 210.82 50.8)
 		)
@@
 		)
 	)
+	(wire
+		(pts
+			(xy 68.58 99.06) (xy 71.12 99.06)
+		)
+		(stroke
+			(width 0)
+			(type default)
+		)
+	)
 	(bus
 		(pts
@@
 	(bus
 		(pts
-			(xy 68.58 111.76) (xy 71.12 111.76)
+			(xy 68.58 114.3) (xy 71.12 114.3)
 		)
 		(stroke
@@
 	(bus
 		(pts
-			(xy 68.58 101.6) (xy 71.12 101.6)
+			(xy 68.58 104.14) (xy 71.12 104.14)
 		)
 		(stroke
@@
 	(bus
 		(pts
-			(xy 68.58 109.22) (xy 71.12 109.22)
+			(xy 68.58 111.76) (xy 71.12 111.76)
 		)
 		(stroke
@@
 	(wire
 		(pts
-			(xy 109.22 172.72) (xy 111.76 172.72)
+			(xy 144.78 35.56) (xy 142.24 35.56)
 		)
 		(stroke
@@
 	(bus
 		(pts
-			(xy 68.58 104.14) (xy 71.12 104.14)
+			(xy 68.58 106.68) (xy 71.12 106.68)
 		)
 		(stroke
@@
 	(wire
 		(pts
+			(xy 142.24 40.64) (xy 144.78 40.64)
+		)
+		(stroke
+			(width 0)
+			(type default)
+		)
+	)
+	(wire
+		(pts
 			(xy 208.28 66.04) (xy 210.82 66.04)
 		)
@@
 	(wire
 		(pts
-			(xy 109.22 170.18) (xy 111.76 170.18)
+			(xy 144.78 38.1) (xy 142.24 38.1)
 		)
 		(stroke
@@
 		)
 	)
-	(label "USBC1_INT#"
-		(at 27.94 106.68 180)
-		(effects
-			(font
-				(size 1.27 1.27)
-			)
-			(justify right bottom)
-		)
-	)
 	(label "WL_REG_ON"
 		(at 190.5 109.22 0)
@@
 	(hierarchical_label "TYPEC1_D"
 		(shape bidirectional)
-		(at 71.12 101.6 0)
+		(at 71.12 104.14 0)
 		(effects
 			(font
@@
 		)
 	)
+	(hierarchical_label "TYPEC1_U2VBUSDET"
+		(shape input)
+		(at 71.12 116.84 0)
+		(effects
+			(font
+				(size 1.27 1.27)
+			)
+			(justify left)
+		)
+	)
 	(hierarchical_label "MAC_RXDV"
 		(shape input)
@@
 		)
 	)
-	(hierarchical_label "TYPEC1_GPIO"
-		(shape input)
-		(at 30.48 106.68 0)
-		(effects
-			(font
-				(size 1.27 1.27)
-			)
-			(justify left)
-		)
-	)
 	(hierarchical_label "GPIO1_C1"
 		(shape output)
@@
 		)
 	)
+	(hierarchical_label "GPIO4_D2"
+		(shape output)
+		(at 231.14 83.82 0)
+		(effects
+			(font
+				(size 1.27 1.27)
+			)
+			(justify left)
+		)
+	)
 	(hierarchical_label "TYPEC0_D"
 		(shape bidirectional)
@@
 	(hierarchical_label "GPIO1_A2"
 		(shape input)
-		(at 109.22 170.18 180)
+		(at 144.78 38.1 0)
 		(effects
 			(font
 				(size 1.27 1.27)
 			)
-			(justify right)
+			(justify left)
 		)
 	)
@@
 		)
 	)
+	(hierarchical_label "GPIO1_A1"
+		(shape input)
+		(at 144.78 40.64 0)
+		(effects
+			(font
+				(size 1.27 1.27)
+			)
+			(justify left)
+		)
+	)
 	(hierarchical_label "DDR0_A"
 		(shape output)
@@
 	(hierarchical_label "TYPEC1_RX"
 		(shape bidirectional)
-		(at 71.12 106.68 0)
+		(at 71.12 109.22 0)
 		(effects
 			(font
@@
 	(hierarchical_label "TYPEC1_AUX_DC"
 		(shape bidirectional)
-		(at 71.12 111.76 0)
+		(at 71.12 114.3 0)
 		(effects
 			(font
@@
 	(hierarchical_label "TYPEC1_TX"
 		(shape output)
-		(at 71.12 104.14 0)
+		(at 71.12 106.68 0)
 		(effects
 			(font
@@
 	(hierarchical_label "GPIO1_A3"
 		(shape output)
-		(at 109.22 172.72 180)
+		(at 144.78 35.56 0)
 		(effects
 			(font
 				(size 1.27 1.27)
 			)
-			(justify right)
+			(justify left)
 		)
 	)
@@
 	(hierarchical_label "TYPEC1_AUX"
 		(shape bidirectional)
-		(at 71.12 109.22 0)
+		(at 71.12 111.76 0)
 		(effects
 			(font
@@
 		)
 	)
+	(hierarchical_label "TYPEC0_U2VBUSDET"
+		(shape input)
+		(at 71.12 99.06 0)
+		(effects
+			(font
+				(size 1.27 1.27)
+			)
+			(justify left)
+		)
+	)
 	(hierarchical_label "GPIO0_A1"
 		(shape output)
@@
 	)
 	(sheet
-		(at 48.26 76.2)
-		(size 20.32 38.1)
+		(at 45.72 76.2)
+		(size 22.86 43.18)
 		(exclude_from_sim no)
 		(in_bom yes)
@@
 		)
 		(property "Sheetname" "CPU-RK3399 USB"
-			(at 48.26 75.4884 0)
+			(at 45.72 75.4884 0)
 			(effects
 				(font
@@
 		)
 		(property "Sheetfile" "CPU-RK3399_USB.kicad_sch"
-			(at 48.26 114.8846 0)
+			(at 45.72 119.9646 0)
 			(effects
 				(font
@@
 		)
 		(pin "TYPEC1_D" bidirectional
-			(at 68.58 101.6 0)
+			(at 68.58 104.14 0)
 			(effects
 				(font
@@
 		)
 		(pin "TYPEC1_TX" output
-			(at 68.58 104.14 0)
+			(at 68.58 106.68 0)
 			(effects
 				(font
@@
 		)
 		(pin "TYPEC1_RX" bidirectional
-			(at 68.58 106.68 0)
+			(at 68.58 109.22 0)
 			(effects
 				(font
@@
 		)
 		(pin "TYPEC1_AUX_DC" bidirectional
-			(at 68.58 111.76 0)
+			(at 68.58 114.3 0)
 			(effects
 				(font
@@
 		)
 		(pin "TYPEC1_AUX" bidirectional
-			(at 68.58 109.22 0)
+			(at 68.58 111.76 0)
+			(effects
+				(font
+					(size 1.27 1.27)
+				)
+				(justify right)
+			)
+		)
+		(pin "TYPEC0_U2VBUSDET" input
+			(at 68.58 99.06 0)
+			(effects
+				(font
+					(size 1.27 1.27)
+				)
+				(justify right)
+			)
+		)
+		(pin "TYPEC1_U2VBUSDET" input
+			(at 68.58 116.84 0)
 			(effects
 				(font
@@
 	(sheet
 		(at 129.54 22.86)
-		(size 12.7 17.78)
+		(size 12.7 20.32)
 		(exclude_from_sim no)
 		(in_bom yes)
@@
 		)
 		(property "Sheetfile" "CPU-RK3399_Protocols.kicad_sch"
-			(at 129.54 41.2246 0)
+			(at 129.54 43.7646 0)
 			(effects
 				(font
@@
 			)
 		)
+		(pin "GPIO1_A3" output
+			(at 142.24 35.56 0)
+			(effects
+				(font
+					(size 1.27 1.27)
+				)
+				(justify right)
+			)
+		)
+		(pin "GPIO1_A2" input
+			(at 142.24 38.1 0)
+			(effects
+				(font
+					(size 1.27 1.27)
+				)
+				(justify right)
+			)
+		)
+		(pin "GPIO1_A1" input
+			(at 142.24 40.64 0)
+			(effects
+				(font
+					(size 1.27 1.27)
+				)
+				(justify right)
+			)
+		)
 		(instances
 			(project "VESA-SBC3399"
@@
 			(effects
 				(font
+					(size 1.27 1.27)
+				)
+				(justify right)
+			)
+		)
+		(pin "GPIO4_D2" output
+			(at 228.6 83.82 0)
+			(effects
+				(font
