File: CPU-RK3399_DVP.kicad_sch (KiCad schematic)
At the start: 1 part, among them U1 RK3399

Commit message: design PMIC
Connections:
- net HDMI_CECINOUT: now reaches U1.AD7 (GPIO4_C7/HDMI_CECINOUT/EDP_HOTPLUG)
Changed lines of the file:
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@@
 		(rev "1.0.0")
 		(company "TickLab")
-		(comment 1 "Project: VESA-SBC3399")
+		(comment 1 "VESA-SBC3399")
 	)
 	(no_connect
@@
 		(at 160.02 111.76)
 	)
+	(wire
+		(pts
+			(xy 63.5 157.48) (xy 78.74 157.48)
+		)
+		(stroke
+			(width 0)
+			(type default)
+		)
+	)
+	(label "HDMI_CEC"
+		(at 66.04 157.48 0)
+		(effects
+			(font
+				(size 1.27 1.27)
+			)
+			(justify left bottom)
+		)
+	)
+	(hierarchical_label "HDMI_CECINOUT"
+		(shape output)
+		(at 63.5 157.48 180)
+		(effects
+			(font
+				(size 1.27 1.27)
+			)
+			(justify right)
+		)
+	)
 	(symbol
-		(lib_name "System On Chip (SoC)/RK3399_1")
 		(lib_id "component_library:System On Chip (SoC)/RK3399")
 		(at 106.68 104.14 0)
@@
 	)
 	(symbol
-		(lib_name "System On Chip (SoC)/RK3399_3")
 		(lib_id "component_library:System On Chip (SoC)/RK3399")
 		(at 182.88 139.7 0)
@@
 	)
 	(symbol
-		(lib_name "System On Chip (SoC)/RK3399_2")
 		(lib_id "component_library:System On Chip (SoC)/RK3399")
 		(at 182.88 104.14 0)
@@
 	)
 	(symbol
-		(lib_name "System On Chip (SoC)/RK3399_4")
 		(lib_id "component_library:System On Chip (SoC)/RK3399")
 		(at 106.68 144.78 0)

Commit message: update design power
Parts:
- renumbered U1 to U2
Changed lines of the file:
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@@
 		(dnp no)
 		(fields_autoplaced yes)
-		(property "Reference" "U1"
+		(property "Reference" "U2"
 			(at 106.68 83.82 0)
 			(effects
@@
 			(project ""
 				(path "/ebc9dc57-8b05-484a-a5cd-c53b1efc71d3/a7299b18-4123-434b-8c69-0b9524fffa12/daf6b753-9b7e-4afa-be48-3492e6b4d132"
-					(reference "U1")
+					(reference "U2")
 					(unit 21)
 				)
@@
 		(dnp no)
 		(fields_autoplaced yes)
-		(property "Reference" "U1"
+		(property "Reference" "U2"
 			(at 182.8761 119.38 0)
 			(effects
@@
 			(project ""
 				(path "/ebc9dc57-8b05-484a-a5cd-c53b1efc71d3/a7299b18-4123-434b-8c69-0b9524fffa12/daf6b753-9b7e-4afa-be48-3492e6b4d132"
-					(reference "U1")
+					(reference "U2")
 					(unit 19)
 				)
@@
 		(dnp no)
 		(fields_autoplaced yes)
-		(property "Reference" "U1"
+		(property "Reference" "U2"
 			(at 182.88 83.82 0)
 			(effects
@@
 			(project ""
 				(path "/ebc9dc57-8b05-484a-a5cd-c53b1efc71d3/a7299b18-4123-434b-8c69-0b9524fffa12/daf6b753-9b7e-4afa-be48-3492e6b4d132"
-					(reference "U1")
+					(reference "U2")
 					(unit 20)
 				)
@@
 		(dnp no)
 		(fields_autoplaced yes)
-		(property "Reference" "U1"
+		(property "Reference" "U2"
 			(at 144.78 38.1 0)
 			(effects
@@
 			(project ""
 				(path "/ebc9dc57-8b05-484a-a5cd-c53b1efc71d3/a7299b18-4123-434b-8c69-0b9524fffa12/daf6b753-9b7e-4afa-be48-3492e6b4d132"
-					(reference "U1")
+					(reference "U2")
 					(unit 28)
 				)
@@
 		(dnp no)
 		(fields_autoplaced yes)
-		(property "Reference" "U1"
+		(property "Reference" "U2"
 			(at 106.68 119.38 0)
 			(effects
@@
 			(project ""
 				(path "/ebc9dc57-8b05-484a-a5cd-c53b1efc71d3/a7299b18-4123-434b-8c69-0b9524fffa12/daf6b753-9b7e-4afa-be48-3492e6b4d132"
-					(reference "U1")
+					(reference "U2")
 					(unit 17)
 				)

Commit message: design DDR
Parts:
- renumbered U2 to U17
Changed lines of the file:
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@@
 		(dnp no)
 		(fields_autoplaced yes)
-		(property "Reference" "U2"
+		(property "Reference" "U17"
 			(at 106.68 83.82 0)
 			(effects
@@
 		)
 		(property "Footprint" "footprints:BGA828C65P31X31_2100X2100X161"
-			(at 109.22 109.22 0)
+			(at 106.68 109.22 0)
 			(effects
 				(font
@@
 			(project ""
 				(path "/ebc9dc57-8b05-484a-a5cd-c53b1efc71d3/a7299b18-4123-434b-8c69-0b9524fffa12/daf6b753-9b7e-4afa-be48-3492e6b4d132"
-					(reference "U2")
+					(reference "U17")
 					(unit 21)
 				)
@@
 		(dnp no)
 		(fields_autoplaced yes)
-		(property "Reference" "U2"
+		(property "Reference" "U17"
 			(at 182.8761 119.38 0)
 			(effects
@@
 		)
 		(property "Footprint" "footprints:BGA828C65P31X31_2100X2100X161"
-			(at 185.42 144.78 0)
+			(at 182.88 144.78 0)
 			(effects
 				(font
@@
 			(project ""
 				(path "/ebc9dc57-8b05-484a-a5cd-c53b1efc71d3/a7299b18-4123-434b-8c69-0b9524fffa12/daf6b753-9b7e-4afa-be48-3492e6b4d132"
-					(reference "U2")
+					(reference "U17")
 					(unit 19)
 				)
@@
 		(dnp no)
 		(fields_autoplaced yes)
-		(property "Reference" "U2"
+		(property "Reference" "U17"
 			(at 182.88 83.82 0)
 			(effects
@@
 		)
 		(property "Footprint" "footprints:BGA828C65P31X31_2100X2100X161"
-			(at 185.42 109.22 0)
+			(at 182.88 109.22 0)
 			(effects
 				(font
@@
 			(project ""
 				(path "/ebc9dc57-8b05-484a-a5cd-c53b1efc71d3/a7299b18-4123-434b-8c69-0b9524fffa12/daf6b753-9b7e-4afa-be48-3492e6b4d132"
-					(reference "U2")
+					(reference "U17")
 					(unit 20)
 				)
@@
 		(dnp no)
 		(fields_autoplaced yes)
-		(property "Reference" "U2"
+		(property "Reference" "U17"
 			(at 144.78 38.1 0)
 			(effects
@@
 		)
 		(property "Footprint" "footprints:BGA828C65P31X31_2100X2100X161"
-			(at 147.32 66.04 0)
+			(at 144.78 66.04 0)
 			(effects
 				(font
@@
 			(project ""
 				(path "/ebc9dc57-8b05-484a-a5cd-c53b1efc71d3/a7299b18-4123-434b-8c69-0b9524fffa12/daf6b753-9b7e-4afa-be48-3492e6b4d132"
-					(reference "U2")
+					(reference "U17")
 					(unit 28)
 				)
@@
 		(dnp no)
 		(fields_autoplaced yes)
-		(property "Reference" "U2"
+		(property "Reference" "U17"
 			(at 106.68 119.38 0)
 			(effects
@@
 		)
 		(property "Footprint" "footprints:BGA828C65P31X31_2100X2100X161"
-			(at 109.22 149.86 0)
+			(at 106.68 149.86 0)
 			(effects
 				(font
@@
 			(project ""
 				(path "/ebc9dc57-8b05-484a-a5cd-c53b1efc71d3/a7299b18-4123-434b-8c69-0b9524fffa12/daf6b753-9b7e-4afa-be48-3492e6b4d132"
-					(reference "U2")
+					(reference "U17")
 					(unit 17)
 				)
