File: CPU-RK3399_HDMI.kicad_sch (KiCad schematic)
At the start: 16 parts, among them U2 RK3399

Commit message: design DDR
Parts:
- renumbered C159 to C286, C160 to C287, C161 to C288, C162 to C289, R52 to R123, R53 to R124, R54 to R125, R55 to R126, R56 to R127, R57 to R128, R58 to R129, R59 to R130, R60 to R131, R61 to R132, U2 to U17
Changed lines of the file:
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@@
 		(on_board yes)
 		(dnp no)
-		(property "Reference" "C159"
+		(property "Reference" "C286"
 			(at 163.83 119.3799 0)
 			(effects
@@
 			(project ""
 				(path "/ebc9dc57-8b05-484a-a5cd-c53b1efc71d3/a7299b18-4123-434b-8c69-0b9524fffa12/25d97e15-4196-4e44-984c-f8c0409a1a6b"
-					(reference "C159")
+					(reference "C286")
 					(unit 1)
 				)
@@
 		(on_board yes)
 		(dnp no)
-		(property "Reference" "#PWR0199"
+		(property "Reference" "#PWR0359"
 			(at 187.96 118.11 0)
 			(effects
@@
 			(project "VESA-SBC3399"
 				(path "/ebc9dc57-8b05-484a-a5cd-c53b1efc71d3/a7299b18-4123-434b-8c69-0b9524fffa12/25d97e15-4196-4e44-984c-f8c0409a1a6b"
-					(reference "#PWR0199")
+					(reference "#PWR0359")
 					(unit 1)
 				)
@@
 		(on_board yes)
 		(dnp no)
-		(property "Reference" "C160"
+		(property "Reference" "C287"
 			(at 176.53 119.3799 0)
 			(effects
@@
 			(project ""
 				(path "/ebc9dc57-8b05-484a-a5cd-c53b1efc71d3/a7299b18-4123-434b-8c69-0b9524fffa12/25d97e15-4196-4e44-984c-f8c0409a1a6b"
-					(reference "C160")
+					(reference "C287")
 					(unit 1)
 				)
@@
 		(on_board yes)
 		(dnp no)
-		(property "Reference" "R59"
+		(property "Reference" "R130"
 			(at 193.04 90.17 0)
 			(effects
@@
 			(project "VESA-SBC3399"
 				(path "/ebc9dc57-8b05-484a-a5cd-c53b1efc71d3/a7299b18-4123-434b-8c69-0b9524fffa12/25d97e15-4196-4e44-984c-f8c0409a1a6b"
-					(reference "R59")
+					(reference "R130")
 					(unit 1)
 				)
@@
 		(on_board yes)
 		(dnp no)
-		(property "Reference" "R52"
+		(property "Reference" "R123"
 			(at 104.14 74.93 0)
 			(effects
@@
 			(project "VESA-SBC3399"
 				(path "/ebc9dc57-8b05-484a-a5cd-c53b1efc71d3/a7299b18-4123-434b-8c69-0b9524fffa12/25d97e15-4196-4e44-984c-f8c0409a1a6b"
-					(reference "R52")
+					(reference "R123")
 					(unit 1)
 				)
@@
 		(dnp no)
 		(fields_autoplaced yes)
-		(property "Reference" "R61"
+		(property "Reference" "R132"
 			(at 127 100.3299 90)
 			(effects
@@
 			(project "VESA-SBC3399"
 				(path "/ebc9dc57-8b05-484a-a5cd-c53b1efc71d3/a7299b18-4123-434b-8c69-0b9524fffa12/25d97e15-4196-4e44-984c-f8c0409a1a6b"
-					(reference "R61")
+					(reference "R132")
 					(unit 1)
 				)
@@
 		(dnp no)
 		(fields_autoplaced yes)
-		(property "Reference" "#PWR0197"
+		(property "Reference" "#PWR0357"
 			(at 124.46 115.57 0)
 			(effects
@@
 			(project "VESA-SBC3399"
 				(path "/ebc9dc57-8b05-484a-a5cd-c53b1efc71d3/a7299b18-4123-434b-8c69-0b9524fffa12/25d97e15-4196-4e44-984c-f8c0409a1a6b"
-					(reference "#PWR0197")
+					(reference "#PWR0357")
 					(unit 1)
 				)
@@
 		(on_board yes)
 		(dnp no)
-		(property "Reference" "#PWR0198"
+		(property "Reference" "#PWR0358"
 			(at 160.02 118.11 0)
 			(effects
@@
 			(project "VESA-SBC3399"
 				(path "/ebc9dc57-8b05-484a-a5cd-c53b1efc71d3/a7299b18-4123-434b-8c69-0b9524fffa12/25d97e15-4196-4e44-984c-f8c0409a1a6b"
-					(reference "#PWR0198")
+					(reference "#PWR0358")
 					(unit 1)
 				)
@@
 		(on_board yes)
 		(dnp no)
-		(property "Reference" "R54"
+		(property "Reference" "R125"
 			(at 193.04 80.01 0)
 			(effects
@@
 			(project "VESA-SBC3399"
 				(path "/ebc9dc57-8b05-484a-a5cd-c53b1efc71d3/a7299b18-4123-434b-8c69-0b9524fffa12/25d97e15-4196-4e44-984c-f8c0409a1a6b"
-					(reference "R54")
+					(reference "R125")
 					(unit 1)
 				)
@@
 		(on_board yes)
 		(dnp no)
-		(property "Reference" "C161"
+		(property "Reference" "C288"
 			(at 191.77 119.3799 0)
 			(effects
@@
 			(project "VESA-SBC3399"
 				(path "/ebc9dc57-8b05-484a-a5cd-c53b1efc71d3/a7299b18-4123-434b-8c69-0b9524fffa12/25d97e15-4196-4e44-984c-f8c0409a1a6b"
-					(reference "C161")
+					(reference "C288")
 					(unit 1)
 				)
@@
 		(dnp no)
 		(fields_autoplaced yes)
-		(property "Reference" "#PWR0201"
+		(property "Reference" "#PWR0361"
 			(at 187.96 138.43 0)
 			(effects
@@
 			(project "VESA-SBC3399"
 				(path "/ebc9dc57-8b05-484a-a5cd-c53b1efc71d3/a7299b18-4123-434b-8c69-0b9524fffa12/25d97e15-4196-4e44-984c-f8c0409a1a6b"
-					(reference "#PWR0201")
+					(reference "#PWR0361")
 					(unit 1)
 				)
@@
 		(on_board yes)
 		(dnp no)
-		(property "Reference" "R56"
+		(property "Reference" "R127"
 			(at 193.04 85.09 0)
 			(effects
@@
 			(project "VESA-SBC3399"
 				(path "/ebc9dc57-8b05-484a-a5cd-c53b1efc71d3/a7299b18-4123-434b-8c69-0b9524fffa12/25d97e15-4196-4e44-984c-f8c0409a1a6b"
-					(reference "R56")
+					(reference "R127")
 					(unit 1)
 				)
@@
 		(on_board yes)
 		(dnp no)
-		(property "Reference" "C162"
+		(property "Reference" "C289"
 			(at 204.47 119.3799 0)
 			(effects
@@
 			(project "VESA-SBC3399"
 				(path "/ebc9dc57-8b05-484a-a5cd-c53b1efc71d3/a7299b18-4123-434b-8c69-0b9524fffa12/25d97e15-4196-4e44-984c-f8c0409a1a6b"
-					(reference "C162")
+					(reference "C289")
 					(unit 1)
 				)
@@
 		(on_board yes)
 		(dnp no)
-		(property "Reference" "#PWR0195"
+		(property "Reference" "#PWR0355"
 			(at 171.45 96.52 0)
 			(effects
@@
 			(project "VESA-SBC3399"
 				(path "/ebc9dc57-8b05-484a-a5cd-c53b1efc71d3/a7299b18-4123-434b-8c69-0b9524fffa12/25d97e15-4196-4e44-984c-f8c0409a1a6b"
-					(reference "#PWR0195")
+					(reference "#PWR0355")
 					(unit 1)
 				)
@@
 		(dnp no)
 		(fields_autoplaced yes)
-		(property "Reference" "U2"
+		(property "Reference" "U17"
 			(at 151.13 68.58 0)
 			(effects
@@
 		)
 		(property "Footprint" "footprints:BGA828C65P31X31_2100X2100X161"
-			(at 152.4 96.52 0)
+			(at 149.86 96.52 0)
 			(effects
 				(font
@@
 			(project ""
 				(path "/ebc9dc57-8b05-484a-a5cd-c53b1efc71d3/a7299b18-4123-434b-8c69-0b9524fffa12/25d97e15-4196-4e44-984c-f8c0409a1a6b"
-					(reference "U2")
+					(reference "U17")
 					(unit 18)
 				)
@@
 		(dnp no)
 		(fields_autoplaced yes)
-		(property "Reference" "#PWR0200"
+		(property "Reference" "#PWR0360"
 			(at 160.02 138.43 0)
 			(effects
@@
 			(project "VESA-SBC3399"
 				(path "/ebc9dc57-8b05-484a-a5cd-c53b1efc71d3/a7299b18-4123-434b-8c69-0b9524fffa12/25d97e15-4196-4e44-984c-f8c0409a1a6b"
-					(reference "#PWR0200")
+					(reference "#PWR0360")
 					(unit 1)
 				)
@@
 		(dnp no)
 		(fields_autoplaced yes)
-		(property "Reference" "R60"
+		(property "Reference" "R131"
 			(at 125.73 85.09 0)
 			(effects
@@
 			(project ""
 				(path "/ebc9dc57-8b05-484a-a5cd-c53b1efc71d3/a7299b18-4123-434b-8c69-0b9524fffa12/25d97e15-4196-4e44-984c-f8c0409a1a6b"
-					(reference "R60")
+					(reference "R131")
 					(unit 1)
 				)
@@
 		(on_board yes)
 		(dnp no)
-		(property "Reference" "R57"
+		(property "Reference" "R128"
 			(at 104.14 87.63 0)
 			(effects
@@
 			(project "VESA-SBC3399"
 				(path "/ebc9dc57-8b05-484a-a5cd-c53b1efc71d3/a7299b18-4123-434b-8c69-0b9524fffa12/25d97e15-4196-4e44-984c-f8c0409a1a6b"
-					(reference "R57")
+					(reference "R128")
 					(unit 1)
 				)
@@
 		(on_board yes)
 		(dnp no)
-		(property "Reference" "R55"
+		(property "Reference" "R126"
 			(at 193.04 82.55 0)
 			(effects
@@
 			(project "VESA-SBC3399"
 				(path "/ebc9dc57-8b05-484a-a5cd-c53b1efc71d3/a7299b18-4123-434b-8c69-0b9524fffa12/25d97e15-4196-4e44-984c-f8c0409a1a6b"
-					(reference "R55")
+					(reference "R126")
 					(unit 1)
 				)
@@
 		(on_board yes)
 		(dnp no)
-		(property "Reference" "#PWR0196"
+		(property "Reference" "#PWR0356"
 			(at 171.45 101.6 0)
 			(effects
@@
 			(project "VESA-SBC3399"
 				(path "/ebc9dc57-8b05-484a-a5cd-c53b1efc71d3/a7299b18-4123-434b-8c69-0b9524fffa12/25d97e15-4196-4e44-984c-f8c0409a1a6b"
-					(reference "#PWR0196")
+					(reference "#PWR0356")
 					(unit 1)
 				)
@@
 		(on_board yes)
 		(dnp no)
-		(property "Reference" "R53"
+		(property "Reference" "R124"
 			(at 193.04 77.47 0)
 			(effects
@@
 			(project ""
 				(path "/ebc9dc57-8b05-484a-a5cd-c53b1efc71d3/a7299b18-4123-434b-8c69-0b9524fffa12/25d97e15-4196-4e44-984c-f8c0409a1a6b"
-					(reference "R53")
+					(reference "R124")
 					(unit 1)
 				)
@@
 		(on_board yes)
 		(dnp no)
-		(property "Reference" "R58"
+		(property "Reference" "R129"
 			(at 193.04 87.63 0)
 			(effects
@@
 			(project "VESA-SBC3399"
 				(path "/ebc9dc57-8b05-484a-a5cd-c53b1efc71d3/a7299b18-4123-434b-8c69-0b9524fffa12/25d97e15-4196-4e44-984c-f8c0409a1a6b"
-					(reference "R58")
+					(reference "R129")
 					(unit 1)
 				)
