File: CPU-RK3399_PCIe.kicad_sch (KiCad schematic)
At the start: 7 parts, among them U1 RK3399

Commit message: design PMIC
Parts:
- removed R51, R52, R53, R54, R55, R56: ~, footprints:RESC1005X35N, symbol component_library:Resistors/0402WGF220JTCE
- removed U1: RK3399, footprints:BGA828C65P31X31_2100X2100X161, symbol component_library:System On Chip (SoC)/RK3399
- added C116, C117: ~, footprints:CAPC1005X50N, symbol component_library:Capacitors/CL05B104KO5NNNC
- added TP7: ~, footprints:, symbol component_library:Mechanical/Test_Point
- added U1: RK3399, footprints:BGA828C65P31X31_2100X2100X161, symbol component_library:System On Chip (SoC)/RK3399
Connections:
- new net: TP7.TP, U1.AE6 (GPIO4_D0/PCIE_CLKREQNB)
- new net +0V9_AVCC: C116.1, U1.W24 (PCIE_AVDD_0V9)
- new net +1V8_VCC: C117.1, U1.Y24 (PCIE_AVDD_1V8)
- new net GND: C116.2, C117.2
- new net PCIe_PER0+: U1.AF30 (PCIE_RX0_P)
- new net PCIe_PER0-: U1.AF31 (PCIE_RX0_N)
- new net PCIe_PER1+: U1.AH30 (PCIE_RX1_P)
- new net PCIe_PER1-: U1.AH31 (PCIE_RX1_N)
- new net PCIe_PER2+: U1.AC27 (PCIE_RX2_P)
- new net PCIe_PER2-: U1.AC28 (PCIE_RX2_N)
- new net PCIe_PER3+: U1.AF27 (PCIE_RX3_P)
- new net PCIe_PER3-: U1.AF28 (PCIE_RX3_N)
- new net PCIe_PET0+: U1.AE30 (PCIE_TX0_P)
- new net PCIe_PET0-: U1.AE31 (PCIE_TX0_N)
- new net PCIe_PET1+: U1.AG30 (PCIE_TX1_P)
- new net PCIe_PET1-: U1.AG31 (PCIE_TX1_N)
- new net PCIe_PET2+: U1.AA27 (PCIE_TX2_P)
- new net PCIe_PET2-: U1.AA28 (PCIE_TX2_N)
- new net PCIe_PET3+: U1.AD27 (PCIE_TX3_P)
- new net PCIe_PET3-: U1.AD28 (PCIE_TX3_N)
- new net PCIe_REFCLK+: U1.AD31 (PCIE_RCLK_100M_P)
- new net PCIe_REFCLK-: U1.AD30 (PCIE_RCLK_100M_N)
- no-connect marks 5 -> 0
Other:
- title: CPU-RK3399 SDIO Controller -> CPU-RK3399 PCIe Controller

Commit message: update design power
Parts:
- renumbered C116 to C119, C117 to C120, TP7 to TP3, U1 to U2
Changed lines of the file:
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@@
 		(on_board yes)
 		(dnp no)
-		(property "Reference" "C117"
+		(property "Reference" "C120"
 			(at 191.77 119.3799 0)
 			(effects
@@
 			(project "VESA-SBC3399"
 				(path "/ebc9dc57-8b05-484a-a5cd-c53b1efc71d3/a7299b18-4123-434b-8c69-0b9524fffa12/8c8e1d96-8c5a-4c87-9cb3-f60d5f431bd8"
-					(reference "C117")
+					(reference "C120")
 					(unit 1)
 				)
@@
 		(on_board yes)
 		(dnp no)
-		(property "Reference" "C116"
+		(property "Reference" "C119"
 			(at 176.53 119.3799 0)
 			(effects
@@
 			(project "VESA-SBC3399"
 				(path "/ebc9dc57-8b05-484a-a5cd-c53b1efc71d3/a7299b18-4123-434b-8c69-0b9524fffa12/8c8e1d96-8c5a-4c87-9cb3-f60d5f431bd8"
-					(reference "C116")
+					(reference "C119")
 					(unit 1)
 				)
@@
 		(dnp no)
 		(fields_autoplaced yes)
-		(property "Reference" "#PWR0144"
+		(property "Reference" "#PWR0131"
 			(at 172.72 135.89 0)
 			(effects
@@
 			(project "VESA-SBC3399"
 				(path "/ebc9dc57-8b05-484a-a5cd-c53b1efc71d3/a7299b18-4123-434b-8c69-0b9524fffa12/8c8e1d96-8c5a-4c87-9cb3-f60d5f431bd8"
-					(reference "#PWR0144")
+					(reference "#PWR0131")
 					(unit 1)
 				)
@@
 		(on_board yes)
 		(dnp no)
-		(property "Reference" "TP7"
+		(property "Reference" "TP3"
 			(at 111.76 96.52 90)
 			(effects
@@
 			(project ""
 				(path "/ebc9dc57-8b05-484a-a5cd-c53b1efc71d3/a7299b18-4123-434b-8c69-0b9524fffa12/8c8e1d96-8c5a-4c87-9cb3-f60d5f431bd8"
-					(reference "TP7")
+					(reference "TP3")
 					(unit 1)
 				)
@@
 		(dnp no)
 		(fields_autoplaced yes)
-		(property "Reference" "U1"
+		(property "Reference" "U2"
 			(at 147.5229 55.88 0)
 			(effects
@@
 			(project ""
 				(path "/ebc9dc57-8b05-484a-a5cd-c53b1efc71d3/a7299b18-4123-434b-8c69-0b9524fffa12/8c8e1d96-8c5a-4c87-9cb3-f60d5f431bd8"
-					(reference "U1")
+					(reference "U2")
 					(unit 8)
 				)
@@
 		(on_board yes)
 		(dnp no)
-		(property "Reference" "#PWR0142"
+		(property "Reference" "#PWR0129"
 			(at 172.72 120.65 0)
 			(effects
@@
 			(project "VESA-SBC3399"
 				(path "/ebc9dc57-8b05-484a-a5cd-c53b1efc71d3/a7299b18-4123-434b-8c69-0b9524fffa12/8c8e1d96-8c5a-4c87-9cb3-f60d5f431bd8"
-					(reference "#PWR0142")
+					(reference "#PWR0129")
 					(unit 1)
 				)
@@
 		(dnp no)
 		(fields_autoplaced yes)
-		(property "Reference" "#PWR0145"
+		(property "Reference" "#PWR0132"
 			(at 187.96 135.89 0)
 			(effects
@@
 			(project "VESA-SBC3399"
 				(path "/ebc9dc57-8b05-484a-a5cd-c53b1efc71d3/a7299b18-4123-434b-8c69-0b9524fffa12/8c8e1d96-8c5a-4c87-9cb3-f60d5f431bd8"
-					(reference "#PWR0145")
+					(reference "#PWR0132")
 					(unit 1)
 				)
@@
 		(on_board yes)
 		(dnp no)
-		(property "Reference" "#PWR0141"
+		(property "Reference" "#PWR0127"
 			(at 168.91 104.14 0)
 			(effects
@@
 			(project "VESA-SBC3399"
 				(path "/ebc9dc57-8b05-484a-a5cd-c53b1efc71d3/a7299b18-4123-434b-8c69-0b9524fffa12/8c8e1d96-8c5a-4c87-9cb3-f60d5f431bd8"
-					(reference "#PWR0141")
+					(reference "#PWR0127")
 					(unit 1)
 				)
@@
 		(on_board yes)
 		(dnp no)
-		(property "Reference" "#PWR0140"
+		(property "Reference" "#PWR0128"
 			(at 168.91 106.68 0)
 			(effects
@@
 			(project "VESA-SBC3399"
 				(path "/ebc9dc57-8b05-484a-a5cd-c53b1efc71d3/a7299b18-4123-434b-8c69-0b9524fffa12/8c8e1d96-8c5a-4c87-9cb3-f60d5f431bd8"
-					(reference "#PWR0140")
+					(reference "#PWR0128")
 					(unit 1)
 				)
@@
 		(on_board yes)
 		(dnp no)
-		(property "Reference" "#PWR0143"
+		(property "Reference" "#PWR0130"
 			(at 187.96 120.65 0)
 			(effects
@@
 			(project "VESA-SBC3399"
 				(path "/ebc9dc57-8b05-484a-a5cd-c53b1efc71d3/a7299b18-4123-434b-8c69-0b9524fffa12/8c8e1d96-8c5a-4c87-9cb3-f60d5f431bd8"
-					(reference "#PWR0143")
+					(reference "#PWR0130")
 					(unit 1)
 				)

Commit message: design DDR
Parts:
- renumbered C119 to C246, C120 to C247, U2 to U17
Changed lines of the file:
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@@
 		(on_board yes)
 		(dnp no)
-		(property "Reference" "C120"
+		(property "Reference" "C247"
 			(at 191.77 119.3799 0)
 			(effects
@@
 			(project "VESA-SBC3399"
 				(path "/ebc9dc57-8b05-484a-a5cd-c53b1efc71d3/a7299b18-4123-434b-8c69-0b9524fffa12/8c8e1d96-8c5a-4c87-9cb3-f60d5f431bd8"
-					(reference "C120")
+					(reference "C247")
 					(unit 1)
 				)
@@
 		(on_board yes)
 		(dnp no)
-		(property "Reference" "C119"
+		(property "Reference" "C246"
 			(at 176.53 119.3799 0)
 			(effects
@@
 			(project "VESA-SBC3399"
 				(path "/ebc9dc57-8b05-484a-a5cd-c53b1efc71d3/a7299b18-4123-434b-8c69-0b9524fffa12/8c8e1d96-8c5a-4c87-9cb3-f60d5f431bd8"
-					(reference "C119")
+					(reference "C246")
 					(unit 1)
 				)
@@
 		(dnp no)
 		(fields_autoplaced yes)
-		(property "Reference" "#PWR0131"
+		(property "Reference" "#PWR0291"
 			(at 172.72 135.89 0)
 			(effects
@@
 			(project "VESA-SBC3399"
 				(path "/ebc9dc57-8b05-484a-a5cd-c53b1efc71d3/a7299b18-4123-434b-8c69-0b9524fffa12/8c8e1d96-8c5a-4c87-9cb3-f60d5f431bd8"
-					(reference "#PWR0131")
+					(reference "#PWR0291")
 					(unit 1)
 				)
@@
 		(dnp no)
 		(fields_autoplaced yes)
-		(property "Reference" "U2"
+		(property "Reference" "U17"
 			(at 147.5229 55.88 0)
 			(effects
@@
 			(project ""
 				(path "/ebc9dc57-8b05-484a-a5cd-c53b1efc71d3/a7299b18-4123-434b-8c69-0b9524fffa12/8c8e1d96-8c5a-4c87-9cb3-f60d5f431bd8"
-					(reference "U2")
+					(reference "U17")
 					(unit 8)
 				)
@@
 		(on_board yes)
 		(dnp no)
-		(property "Reference" "#PWR0129"
+		(property "Reference" "#PWR0289"
 			(at 172.72 120.65 0)
 			(effects
@@
 			(project "VESA-SBC3399"
 				(path "/ebc9dc57-8b05-484a-a5cd-c53b1efc71d3/a7299b18-4123-434b-8c69-0b9524fffa12/8c8e1d96-8c5a-4c87-9cb3-f60d5f431bd8"
-					(reference "#PWR0129")
+					(reference "#PWR0289")
 					(unit 1)
 				)
@@
 		(dnp no)
 		(fields_autoplaced yes)
-		(property "Reference" "#PWR0132"
+		(property "Reference" "#PWR0292"
 			(at 187.96 135.89 0)
 			(effects
@@
 			(project "VESA-SBC3399"
 				(path "/ebc9dc57-8b05-484a-a5cd-c53b1efc71d3/a7299b18-4123-434b-8c69-0b9524fffa12/8c8e1d96-8c5a-4c87-9cb3-f60d5f431bd8"
-					(reference "#PWR0132")
+					(reference "#PWR0292")
 					(unit 1)
 				)
@@
 		(on_board yes)
 		(dnp no)
-		(property "Reference" "#PWR0127"
+		(property "Reference" "#PWR0287"
 			(at 168.91 104.14 0)
 			(effects
@@
 			(project "VESA-SBC3399"
 				(path "/ebc9dc57-8b05-484a-a5cd-c53b1efc71d3/a7299b18-4123-434b-8c69-0b9524fffa12/8c8e1d96-8c5a-4c87-9cb3-f60d5f431bd8"
-					(reference "#PWR0127")
+					(reference "#PWR0287")
 					(unit 1)
 				)
@@
 		(on_board yes)
 		(dnp no)
-		(property "Reference" "#PWR0128"
+		(property "Reference" "#PWR0288"
 			(at 168.91 106.68 0)
 			(effects
@@
 			(project "VESA-SBC3399"
 				(path "/ebc9dc57-8b05-484a-a5cd-c53b1efc71d3/a7299b18-4123-434b-8c69-0b9524fffa12/8c8e1d96-8c5a-4c87-9cb3-f60d5f431bd8"
-					(reference "#PWR0128")
+					(reference "#PWR0288")
 					(unit 1)
 				)
@@
 		(on_board yes)
 		(dnp no)
-		(property "Reference" "#PWR0130"
+		(property "Reference" "#PWR0290"
 			(at 187.96 120.65 0)
 			(effects
@@
 			(project "VESA-SBC3399"
 				(path "/ebc9dc57-8b05-484a-a5cd-c53b1efc71d3/a7299b18-4123-434b-8c69-0b9524fffa12/8c8e1d96-8c5a-4c87-9cb3-f60d5f431bd8"
-					(reference "#PWR0130")
+					(reference "#PWR0290")
 					(unit 1)
 				)
