File: CPU-RK3399_PMU_Controller.kicad_sch (KiCad schematic)
At the start: 15 parts, among them U1 RK3399

Commit message: design PMIC
Parts:
- added Q2: ~, footprints:, symbol component_library:FETs/WNM2021-3/TR
- added R61: ~, footprints:RESC1005X35N, symbol component_library:Resistors/0402WGF0000TCE
Connections:
- net GPIO4_D2: now reaches U1.AH3 (GPIO4_D2)
- net GPIO4_D4: now reaches U1.AH5 (GPIO4_D4)
- net GPIO4_C5: now reaches U1.AK1 (GPIO4_C5/SPDIF_TX)
- net GPIO4_D3: now reaches U1.AK3 (GPIO4_D3)
- net ???DP_PWR: now reaches U1.L25 (GPIO1_C6/TCPD_VBUS_SOURCE0)
- net GPIO1_D0: now reaches U1.L26 (GPIO1_D0/TCPD_VBUS_SOURCE2)
- net at U1.M31 (GPIO1_C7/TCPD_VBUS_SOURCE1): now also Q2.S (Source), R61.1
- new net +1V8_VCC: Q2.G (Gate)
- new net GPIO1_C7: Q2.D (Drain), R61.2
- no-connect marks 10 -> 15
Other:
- moved on the sheet: C60, C62, R2, R3, Y1

Commit message: update design power
Parts:
- renumbered C59 to C112, C60 to C113, C61 to C114, C62 to C115, C63 to C116, Q2 to Q3, R1 to R17, R2 to R18, R3 to R19, R61 to R20, R4 to R21, R5 to R22, R6 to R23, U1 to U2, Y1 to Y2
Changed lines of the file:
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@@
 		(on_board yes)
 		(dnp no)
-		(property "Reference" "R61"
+		(property "Reference" "R20"
 			(at 214.63 110.49 0)
 			(effects
@@
 			(project ""
 				(path "/ebc9dc57-8b05-484a-a5cd-c53b1efc71d3/a7299b18-4123-434b-8c69-0b9524fffa12/8f828ad1-c2b0-4246-8b6b-a40b1b5d18bf"
-					(reference "R61")
+					(reference "R20")
 					(unit 1)
 				)
@@
 		(dnp no)
 		(fields_autoplaced yes)
-		(property "Reference" "#PWR031"
+		(property "Reference" "#PWR0112"
 			(at 78.74 54.61 0)
 			(effects
@@
 			(project "VESA-SBC3399"
 				(path "/ebc9dc57-8b05-484a-a5cd-c53b1efc71d3/a7299b18-4123-434b-8c69-0b9524fffa12/8f828ad1-c2b0-4246-8b6b-a40b1b5d18bf"
-					(reference "#PWR031")
+					(reference "#PWR0112")
 					(unit 1)
 				)
@@
 		(on_board yes)
 		(dnp yes)
-		(property "Reference" "C61"
+		(property "Reference" "C114"
 			(at 229.87 58.4199 0)
 			(effects
@@
 			(project "VESA-SBC3399"
 				(path "/ebc9dc57-8b05-484a-a5cd-c53b1efc71d3/a7299b18-4123-434b-8c69-0b9524fffa12/8f828ad1-c2b0-4246-8b6b-a40b1b5d18bf"
-					(reference "C61")
+					(reference "C114")
 					(unit 1)
 				)
@@
 		(dnp no)
 		(fields_autoplaced yes)
-		(property "Reference" "#PWR036"
+		(property "Reference" "#PWR0117"
 			(at 91.44 125.73 0)
 			(effects
@@
 			(project "VESA-SBC3399"
 				(path "/ebc9dc57-8b05-484a-a5cd-c53b1efc71d3/a7299b18-4123-434b-8c69-0b9524fffa12/8f828ad1-c2b0-4246-8b6b-a40b1b5d18bf"
-					(reference "#PWR036")
+					(reference "#PWR0117")
 					(unit 1)
 				)
@@
 		(dnp no)
 		(fields_autoplaced yes)
-		(property "Reference" "#PWR038"
+		(property "Reference" "#PWR0119"
 			(at 269.24 158.75 0)
 			(effects
@@
 			(project "VESA-SBC3399"
 				(path "/ebc9dc57-8b05-484a-a5cd-c53b1efc71d3/a7299b18-4123-434b-8c69-0b9524fffa12/8f828ad1-c2b0-4246-8b6b-a40b1b5d18bf"
-					(reference "#PWR038")
+					(reference "#PWR0119")
 					(unit 1)
 				)
@@
 		(dnp no)
 		(fields_autoplaced yes)
-		(property "Reference" "U1"
+		(property "Reference" "U2"
 			(at 139.7 45.72 0)
 			(effects
@@
 			(project ""
 				(path "/ebc9dc57-8b05-484a-a5cd-c53b1efc71d3/a7299b18-4123-434b-8c69-0b9524fffa12/8f828ad1-c2b0-4246-8b6b-a40b1b5d18bf"
-					(reference "U1")
+					(reference "U2")
 					(unit 11)
 				)
@@
 		(dnp no)
 		(fields_autoplaced yes)
-		(property "Reference" "#PWR033"
+		(property "Reference" "#PWR0114"
 			(at 40.64 80.01 0)
 			(effects
@@
 			(project "VESA-SBC3399"
 				(path "/ebc9dc57-8b05-484a-a5cd-c53b1efc71d3/a7299b18-4123-434b-8c69-0b9524fffa12/8f828ad1-c2b0-4246-8b6b-a40b1b5d18bf"
-					(reference "#PWR033")
+					(reference "#PWR0114")
 					(unit 1)
 				)
@@
 		(dnp no)
 		(fields_autoplaced yes)
-		(property "Reference" "R4"
+		(property "Reference" "R21"
 			(at 78.74 107.9499 90)
 			(effects
@@
 			(project "VESA-SBC3399"
 				(path "/ebc9dc57-8b05-484a-a5cd-c53b1efc71d3/a7299b18-4123-434b-8c69-0b9524fffa12/8f828ad1-c2b0-4246-8b6b-a40b1b5d18bf"
-					(reference "R4")
+					(reference "R21")
 					(unit 1)
 				)
@@
 		(dnp no)
 		(fields_autoplaced yes)
-		(property "Reference" "R1"
+		(property "Reference" "R17"
 			(at 234.95 46.99 0)
 			(effects
@@
 			(project ""
 				(path "/ebc9dc57-8b05-484a-a5cd-c53b1efc71d3/a7299b18-4123-434b-8c69-0b9524fffa12/8f828ad1-c2b0-4246-8b6b-a40b1b5d18bf"
-					(reference "R1")
+					(reference "R17")
 					(unit 1)
 				)
@@
 		(dnp yes)
 		(fields_autoplaced yes)
-		(property "Reference" "R5"
+		(property "Reference" "R22"
 			(at 271.78 130.8099 90)
 			(effects
@@
 			(project ""
 				(path "/ebc9dc57-8b05-484a-a5cd-c53b1efc71d3/a7299b18-4123-434b-8c69-0b9524fffa12/8f828ad1-c2b0-4246-8b6b-a40b1b5d18bf"
-					(reference "R5")
+					(reference "R22")
 					(unit 1)
 				)
@@
 		(dnp no)
 		(fields_autoplaced yes)
-		(property "Reference" "R2"
+		(property "Reference" "R18"
 			(at 71.12 62.2299 90)
 			(effects
@@
 			(project "VESA-SBC3399"
 				(path "/ebc9dc57-8b05-484a-a5cd-c53b1efc71d3/a7299b18-4123-434b-8c69-0b9524fffa12/8f828ad1-c2b0-4246-8b6b-a40b1b5d18bf"
-					(reference "R2")
+					(reference "R18")
 					(unit 1)
 				)
@@
 		(dnp yes)
 		(fields_autoplaced yes)
-		(property "Reference" "Q2"
+		(property "Reference" "Q3"
 			(at 214.63 99.06 90)
 			(effects
@@
 			(project ""
 				(path "/ebc9dc57-8b05-484a-a5cd-c53b1efc71d3/a7299b18-4123-434b-8c69-0b9524fffa12/8f828ad1-c2b0-4246-8b6b-a40b1b5d18bf"
-					(reference "Q2")
+					(reference "Q3")
 					(unit 1)
 				)
@@
 		(on_board yes)
 		(dnp no)
-		(property "Reference" "C60"
+		(property "Reference" "C113"
 			(at 49.53 45.72 90)
 			(effects
@@
 			(project "VESA-SBC3399"
 				(path "/ebc9dc57-8b05-484a-a5cd-c53b1efc71d3/a7299b18-4123-434b-8c69-0b9524fffa12/8f828ad1-c2b0-4246-8b6b-a40b1b5d18bf"
-					(reference "C60")
+					(reference "C113")
 					(unit 1)
 				)
@@
 		(dnp no)
 		(fields_autoplaced yes)
-		(property "Reference" "Y1"
+		(property "Reference" "Y2"
 			(at 58.42 62.2299 90)
 			(effects
@@
 			(project "VESA-SBC3399"
 				(path "/ebc9dc57-8b05-484a-a5cd-c53b1efc71d3/a7299b18-4123-434b-8c69-0b9524fffa12/8f828ad1-c2b0-4246-8b6b-a40b1b5d18bf"
-					(reference "Y1")
+					(reference "Y2")
 					(unit 1)
 				)
@@
 		(on_board yes)
 		(dnp no)
-		(property "Reference" "C62"
+		(property "Reference" "C115"
 			(at 49.53 83.82 90)
 			(effects
@@
 			(project ""
 				(path "/ebc9dc57-8b05-484a-a5cd-c53b1efc71d3/a7299b18-4123-434b-8c69-0b9524fffa12/8f828ad1-c2b0-4246-8b6b-a40b1b5d18bf"
-					(reference "C62")
+					(reference "C115")
 					(unit 1)
 				)
@@
 		(dnp no)
 		(fields_autoplaced yes)
-		(property "Reference" "#PWR032"
+		(property "Reference" "#PWR0113"
 			(at 226.06 74.93 0)
 			(effects
@@
 			(project "VESA-SBC3399"
 				(path "/ebc9dc57-8b05-484a-a5cd-c53b1efc71d3/a7299b18-4123-434b-8c69-0b9524fffa12/8f828ad1-c2b0-4246-8b6b-a40b1b5d18bf"
-					(reference "#PWR032")
+					(reference "#PWR0113")
 					(unit 1)
 				)
@@
 		(on_board yes)
 		(dnp no)
-		(property "Reference" "C63"
+		(property "Reference" "C116"
 			(at 95.25 106.6799 0)
 			(effects
@@
 			(project "VESA-SBC3399"
 				(path "/ebc9dc57-8b05-484a-a5cd-c53b1efc71d3/a7299b18-4123-434b-8c69-0b9524fffa12/8f828ad1-c2b0-4246-8b6b-a40b1b5d18bf"
-					(reference "C63")
+					(reference "C116")
 					(unit 1)
 				)
@@
 		(on_board yes)
 		(dnp no)
-		(property "Reference" "#PWR037"
+		(property "Reference" "#PWR0118"
 			(at 269.24 130.81 0)
 			(effects
@@
 			(project "VESA-SBC3399"
 				(path "/ebc9dc57-8b05-484a-a5cd-c53b1efc71d3/a7299b18-4123-434b-8c69-0b9524fffa12/8f828ad1-c2b0-4246-8b6b-a40b1b5d18bf"
-					(reference "#PWR037")
+					(reference "#PWR0118")
 					(unit 1)
 				)
@@
 		(on_board yes)
 		(dnp no)
-		(property "Reference" "C59"
+		(property "Reference" "C112"
 			(at 82.55 38.0999 0)
 			(effects
@@
 			(project ""
 				(path "/ebc9dc57-8b05-484a-a5cd-c53b1efc71d3/a7299b18-4123-434b-8c69-0b9524fffa12/8f828ad1-c2b0-4246-8b6b-a40b1b5d18bf"
-					(reference "C59")
+					(reference "C112")
 					(unit 1)
 				)
@@
 		(dnp yes)
 		(fields_autoplaced yes)
-		(property "Reference" "R6"
+		(property "Reference" "R23"
 			(at 271.78 143.5099 90)
 			(effects
@@
 			(project ""
 				(path "/ebc9dc57-8b05-484a-a5cd-c53b1efc71d3/a7299b18-4123-434b-8c69-0b9524fffa12/8f828ad1-c2b0-4246-8b6b-a40b1b5d18bf"
-					(reference "R6")
+					(reference "R23")
 					(unit 1)
 				)
@@
 		(on_board yes)
 		(dnp no)
-		(property "Reference" "#PWR0132"
+		(property "Reference" "#PWR0115"
 			(at 213.36 92.71 0)
 			(effects
@@
 			(project "VESA-SBC3399"
 				(path "/ebc9dc57-8b05-484a-a5cd-c53b1efc71d3/a7299b18-4123-434b-8c69-0b9524fffa12/8f828ad1-c2b0-4246-8b6b-a40b1b5d18bf"
-					(reference "#PWR0132")
+					(reference "#PWR0115")
 					(unit 1)
 				)
@@
 		(on_board yes)
 		(dnp no)
-		(property "Reference" "#PWR035"
+		(property "Reference" "#PWR0116"
 			(at 91.44 105.41 0)
 			(effects
@@
 			(project "VESA-SBC3399"
 				(path "/ebc9dc57-8b05-484a-a5cd-c53b1efc71d3/a7299b18-4123-434b-8c69-0b9524fffa12/8f828ad1-c2b0-4246-8b6b-a40b1b5d18bf"
-					(reference "#PWR035")
+					(reference "#PWR0116")
 					(unit 1)
 				)
@@
 		(on_board yes)
 		(dnp no)
-		(property "Reference" "R3"
+		(property "Reference" "R19"
 			(at 62.23 80.01 0)
 			(effects
@@
 			(project "VESA-SBC3399"
 				(path "/ebc9dc57-8b05-484a-a5cd-c53b1efc71d3/a7299b18-4123-434b-8c69-0b9524fffa12/8f828ad1-c2b0-4246-8b6b-a40b1b5d18bf"
-					(reference "R3")
+					(reference "R19")
 					(unit 1)
 				)

Commit message: design DDR
Parts:
- renumbered C112 to C239, C113 to C240, C114 to C241, C115 to C242, C116 to C243, R17 to R88, R18 to R89, R19 to R90, R20 to R91, R21 to R92, R22 to R93, R23 to R94, U2 to U17
Changed lines of the file:
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@@
 		(on_board yes)
 		(dnp no)
-		(property "Reference" "R20"
+		(property "Reference" "R91"
 			(at 214.63 110.49 0)
 			(effects
@@
 			(project ""
 				(path "/ebc9dc57-8b05-484a-a5cd-c53b1efc71d3/a7299b18-4123-434b-8c69-0b9524fffa12/8f828ad1-c2b0-4246-8b6b-a40b1b5d18bf"
-					(reference "R20")
+					(reference "R91")
 					(unit 1)
 				)
@@
 		(dnp no)
 		(fields_autoplaced yes)
-		(property "Reference" "#PWR0112"
+		(property "Reference" "#PWR0272"
 			(at 78.74 54.61 0)
 			(effects
@@
 			(project "VESA-SBC3399"
 				(path "/ebc9dc57-8b05-484a-a5cd-c53b1efc71d3/a7299b18-4123-434b-8c69-0b9524fffa12/8f828ad1-c2b0-4246-8b6b-a40b1b5d18bf"
-					(reference "#PWR0112")
+					(reference "#PWR0272")
 					(unit 1)
 				)
@@
 		(on_board yes)
 		(dnp yes)
-		(property "Reference" "C114"
+		(property "Reference" "C241"
 			(at 229.87 58.4199 0)
 			(effects
@@
 			(project "VESA-SBC3399"
 				(path "/ebc9dc57-8b05-484a-a5cd-c53b1efc71d3/a7299b18-4123-434b-8c69-0b9524fffa12/8f828ad1-c2b0-4246-8b6b-a40b1b5d18bf"
-					(reference "C114")
+					(reference "C241")
 					(unit 1)
 				)
@@
 		(dnp no)
 		(fields_autoplaced yes)
-		(property "Reference" "#PWR0117"
+		(property "Reference" "#PWR0277"
 			(at 91.44 125.73 0)
 			(effects
@@
 			(project "VESA-SBC3399"
 				(path "/ebc9dc57-8b05-484a-a5cd-c53b1efc71d3/a7299b18-4123-434b-8c69-0b9524fffa12/8f828ad1-c2b0-4246-8b6b-a40b1b5d18bf"
-					(reference "#PWR0117")
+					(reference "#PWR0277")
 					(unit 1)
 				)
@@
 		(dnp no)
 		(fields_autoplaced yes)
-		(property "Reference" "#PWR0119"
+		(property "Reference" "#PWR0279"
 			(at 269.24 158.75 0)
 			(effects
@@
 			(project "VESA-SBC3399"
 				(path "/ebc9dc57-8b05-484a-a5cd-c53b1efc71d3/a7299b18-4123-434b-8c69-0b9524fffa12/8f828ad1-c2b0-4246-8b6b-a40b1b5d18bf"
-					(reference "#PWR0119")
+					(reference "#PWR0279")
 					(unit 1)
 				)
@@
 		(dnp no)
 		(fields_autoplaced yes)
-		(property "Reference" "U2"
+		(property "Reference" "U17"
 			(at 139.7 45.72 0)
 			(effects
@@
 		)
 		(property "Footprint" "footprints:BGA828C65P31X31_2100X2100X161"
-			(at 157.48 88.9 0)
+			(at 139.7 88.9 0)
 			(effects
 				(font
@@
 			(project ""
 				(path "/ebc9dc57-8b05-484a-a5cd-c53b1efc71d3/a7299b18-4123-434b-8c69-0b9524fffa12/8f828ad1-c2b0-4246-8b6b-a40b1b5d18bf"
-					(reference "U2")
+					(reference "U17")
 					(unit 11)
 				)
@@
 		(dnp no)
 		(fields_autoplaced yes)
-		(property "Reference" "#PWR0114"
+		(property "Reference" "#PWR0274"
 			(at 40.64 80.01 0)
 			(effects
@@
 			(project "VESA-SBC3399"
 				(path "/ebc9dc57-8b05-484a-a5cd-c53b1efc71d3/a7299b18-4123-434b-8c69-0b9524fffa12/8f828ad1-c2b0-4246-8b6b-a40b1b5d18bf"
-					(reference "#PWR0114")
+					(reference "#PWR0274")
 					(unit 1)
 				)
@@
 		(dnp no)
 		(fields_autoplaced yes)
-		(property "Reference" "R21"
+		(property "Reference" "R92"
 			(at 78.74 107.9499 90)
 			(effects
@@
 			(project "VESA-SBC3399"
 				(path "/ebc9dc57-8b05-484a-a5cd-c53b1efc71d3/a7299b18-4123-434b-8c69-0b9524fffa12/8f828ad1-c2b0-4246-8b6b-a40b1b5d18bf"
-					(reference "R21")
+					(reference "R92")
 					(unit 1)
 				)
@@
 		(dnp no)
 		(fields_autoplaced yes)
-		(property "Reference" "R17"
+		(property "Reference" "R88"
 			(at 234.95 46.99 0)
 			(effects
@@
 			(project ""
 				(path "/ebc9dc57-8b05-484a-a5cd-c53b1efc71d3/a7299b18-4123-434b-8c69-0b9524fffa12/8f828ad1-c2b0-4246-8b6b-a40b1b5d18bf"
-					(reference "R17")
+					(reference "R88")
 					(unit 1)
 				)
@@
 		(dnp yes)
 		(fields_autoplaced yes)
-		(property "Reference" "R22"
+		(property "Reference" "R93"
 			(at 271.78 130.8099 90)
 			(effects
@@
 			(project ""
 				(path "/ebc9dc57-8b05-484a-a5cd-c53b1efc71d3/a7299b18-4123-434b-8c69-0b9524fffa12/8f828ad1-c2b0-4246-8b6b-a40b1b5d18bf"
-					(reference "R22")
+					(reference "R93")
 					(unit 1)
 				)
@@
 		(dnp no)
 		(fields_autoplaced yes)
-		(property "Reference" "R18"
+		(property "Reference" "R89"
 			(at 71.12 62.2299 90)
 			(effects
@@
 			(project "VESA-SBC3399"
 				(path "/ebc9dc57-8b05-484a-a5cd-c53b1efc71d3/a7299b18-4123-434b-8c69-0b9524fffa12/8f828ad1-c2b0-4246-8b6b-a40b1b5d18bf"
-					(reference "R18")
+					(reference "R89")
 					(unit 1)
 				)
@@
 		(on_board yes)
 		(dnp no)
-		(property "Reference" "C113"
+		(property "Reference" "C240"
 			(at 49.53 45.72 90)
 			(effects
@@
 			(project "VESA-SBC3399"
 				(path "/ebc9dc57-8b05-484a-a5cd-c53b1efc71d3/a7299b18-4123-434b-8c69-0b9524fffa12/8f828ad1-c2b0-4246-8b6b-a40b1b5d18bf"
-					(reference "C113")
+					(reference "C240")
 					(unit 1)
 				)
@@
 		(on_board yes)
 		(dnp no)
-		(property "Reference" "C115"
+		(property "Reference" "C242"
 			(at 49.53 83.82 90)
 			(effects
@@
 			(project ""
 				(path "/ebc9dc57-8b05-484a-a5cd-c53b1efc71d3/a7299b18-4123-434b-8c69-0b9524fffa12/8f828ad1-c2b0-4246-8b6b-a40b1b5d18bf"
-					(reference "C115")
+					(reference "C242")
 					(unit 1)
 				)
@@
 		(dnp no)
 		(fields_autoplaced yes)
-		(property "Reference" "#PWR0113"
+		(property "Reference" "#PWR0273"
 			(at 226.06 74.93 0)
 			(effects
@@
 			(project "VESA-SBC3399"
 				(path "/ebc9dc57-8b05-484a-a5cd-c53b1efc71d3/a7299b18-4123-434b-8c69-0b9524fffa12/8f828ad1-c2b0-4246-8b6b-a40b1b5d18bf"
-					(reference "#PWR0113")
+					(reference "#PWR0273")
 					(unit 1)
 				)
@@
 		(on_board yes)
 		(dnp no)
-		(property "Reference" "C116"
+		(property "Reference" "C243"
 			(at 95.25 106.6799 0)
 			(effects
@@
 			(project "VESA-SBC3399"
 				(path "/ebc9dc57-8b05-484a-a5cd-c53b1efc71d3/a7299b18-4123-434b-8c69-0b9524fffa12/8f828ad1-c2b0-4246-8b6b-a40b1b5d18bf"
-					(reference "C116")
+					(reference "C243")
 					(unit 1)
 				)
@@
 		(on_board yes)
 		(dnp no)
-		(property "Reference" "#PWR0118"
+		(property "Reference" "#PWR0278"
 			(at 269.24 130.81 0)
 			(effects
@@
 			(project "VESA-SBC3399"
 				(path "/ebc9dc57-8b05-484a-a5cd-c53b1efc71d3/a7299b18-4123-434b-8c69-0b9524fffa12/8f828ad1-c2b0-4246-8b6b-a40b1b5d18bf"
-					(reference "#PWR0118")
+					(reference "#PWR0278")
 					(unit 1)
 				)
@@
 		(on_board yes)
 		(dnp no)
-		(property "Reference" "C112"
+		(property "Reference" "C239"
 			(at 82.55 38.0999 0)
 			(effects
@@
 			(project ""
 				(path "/ebc9dc57-8b05-484a-a5cd-c53b1efc71d3/a7299b18-4123-434b-8c69-0b9524fffa12/8f828ad1-c2b0-4246-8b6b-a40b1b5d18bf"
-					(reference "C112")
+					(reference "C239")
 					(unit 1)
 				)
@@
 		(dnp yes)
 		(fields_autoplaced yes)
-		(property "Reference" "R23"
+		(property "Reference" "R94"
 			(at 271.78 143.5099 90)
 			(effects
@@
 			(project ""
 				(path "/ebc9dc57-8b05-484a-a5cd-c53b1efc71d3/a7299b18-4123-434b-8c69-0b9524fffa12/8f828ad1-c2b0-4246-8b6b-a40b1b5d18bf"
-					(reference "R23")
+					(reference "R94")
 					(unit 1)
 				)
@@
 		(on_board yes)
 		(dnp no)
-		(property "Reference" "#PWR0115"
+		(property "Reference" "#PWR0275"
 			(at 213.36 92.71 0)
 			(effects
@@
 			(project "VESA-SBC3399"
 				(path "/ebc9dc57-8b05-484a-a5cd-c53b1efc71d3/a7299b18-4123-434b-8c69-0b9524fffa12/8f828ad1-c2b0-4246-8b6b-a40b1b5d18bf"
-					(reference "#PWR0115")
+					(reference "#PWR0275")
 					(unit 1)
 				)
@@
 		(on_board yes)
 		(dnp no)
-		(property "Reference" "#PWR0116"
+		(property "Reference" "#PWR0276"
 			(at 91.44 105.41 0)
 			(effects
@@
 			(project "VESA-SBC3399"
 				(path "/ebc9dc57-8b05-484a-a5cd-c53b1efc71d3/a7299b18-4123-434b-8c69-0b9524fffa12/8f828ad1-c2b0-4246-8b6b-a40b1b5d18bf"
-					(reference "#PWR0116")
+					(reference "#PWR0276")
 					(unit 1)
 				)
@@
 		(on_board yes)
 		(dnp no)
-		(property "Reference" "R19"
+		(property "Reference" "R90"
 			(at 62.23 80.01 0)
 			(effects
@@
 			(project "VESA-SBC3399"
 				(path "/ebc9dc57-8b05-484a-a5cd-c53b1efc71d3/a7299b18-4123-434b-8c69-0b9524fffa12/8f828ad1-c2b0-4246-8b6b-a40b1b5d18bf"
-					(reference "R19")
+					(reference "R90")
 					(unit 1)
 				)
