File: CPU-RK3399_Protocols.kicad_sch (KiCad schematic)
At the start: 10 parts, among them U1 RK3399

Commit message: update design power
Parts:
- renumbered Q1 to Q4, R63 to R73, R62 to R74, R58 to R75, R57 to R76, R59 to R77, R60 to R78, TP5 to TP7, U1 to U2
Changed lines of the file:
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@@
 		(dnp no)
 		(fields_autoplaced yes)
-		(property "Reference" "U1"
+		(property "Reference" "U2"
 			(at 248.9182 30.48 0)
 			(effects
@@
 			(project "VESA-SBC3399"
 				(path "/ebc9dc57-8b05-484a-a5cd-c53b1efc71d3/a7299b18-4123-434b-8c69-0b9524fffa12/6aed072b-e48f-49d3-9ccf-1a1784592333"
-					(reference "U1")
+					(reference "U2")
 					(unit 32)
 				)
@@
 		(dnp yes)
 		(fields_autoplaced yes)
-		(property "Reference" "R62"
+		(property "Reference" "R74"
 			(at 154.94 46.9899 90)
 			(effects
@@
 			(project "VESA-SBC3399"
 				(path "/ebc9dc57-8b05-484a-a5cd-c53b1efc71d3/a7299b18-4123-434b-8c69-0b9524fffa12/6aed072b-e48f-49d3-9ccf-1a1784592333"
-					(reference "R62")
+					(reference "R74")
 					(unit 1)
 				)
@@
 		(dnp yes)
 		(fields_autoplaced yes)
-		(property "Reference" "R57"
+		(property "Reference" "R76"
 			(at 91.44 100.3299 90)
 			(effects
@@
 			(project "VESA-SBC3399"
 				(path "/ebc9dc57-8b05-484a-a5cd-c53b1efc71d3/a7299b18-4123-434b-8c69-0b9524fffa12/6aed072b-e48f-49d3-9ccf-1a1784592333"
-					(reference "R57")
+					(reference "R76")
 					(unit 1)
 				)
@@
 		(on_board yes)
 		(dnp no)
-		(property "Reference" "TP5"
+		(property "Reference" "TP7"
 			(at 177.8 111.76 90)
 			(effects
@@
 			(project "VESA-SBC3399"
 				(path "/ebc9dc57-8b05-484a-a5cd-c53b1efc71d3/a7299b18-4123-434b-8c69-0b9524fffa12/6aed072b-e48f-49d3-9ccf-1a1784592333"
-					(reference "TP5")
+					(reference "TP7")
 					(unit 1)
 				)
@@
 		(on_board yes)
 		(dnp no)
-		(property "Reference" "#PWR0133"
+		(property "Reference" "#PWR0204"
 			(at 157.48 44.45 0)
 			(effects
@@
 			(project "VESA-SBC3399"
 				(path "/ebc9dc57-8b05-484a-a5cd-c53b1efc71d3/a7299b18-4123-434b-8c69-0b9524fffa12/6aed072b-e48f-49d3-9ccf-1a1784592333"
-					(reference "#PWR0133")
+					(reference "#PWR0204")
 					(unit 1)
 				)
@@
 		(dnp yes)
 		(fields_autoplaced yes)
-		(property "Reference" "R59"
+		(property "Reference" "R77"
 			(at 81.28 140.9699 90)
 			(effects
@@
 			(project "VESA-SBC3399"
 				(path "/ebc9dc57-8b05-484a-a5cd-c53b1efc71d3/a7299b18-4123-434b-8c69-0b9524fffa12/6aed072b-e48f-49d3-9ccf-1a1784592333"
-					(reference "R59")
+					(reference "R77")
 					(unit 1)
 				)
@@
 		(on_board yes)
 		(dnp no)
-		(property "Reference" "Q1"
+		(property "Reference" "Q4"
 			(at 44.4499 120.65 0)
 			(effects
@@
 			(project "VESA-SBC3399"
 				(path "/ebc9dc57-8b05-484a-a5cd-c53b1efc71d3/a7299b18-4123-434b-8c69-0b9524fffa12/6aed072b-e48f-49d3-9ccf-1a1784592333"
-					(reference "Q1")
+					(reference "Q4")
 					(unit 1)
 				)
@@
 		(dnp yes)
 		(fields_autoplaced yes)
-		(property "Reference" "R60"
+		(property "Reference" "R78"
 			(at 91.44 140.9699 90)
 			(effects
@@
 			(project "VESA-SBC3399"
 				(path "/ebc9dc57-8b05-484a-a5cd-c53b1efc71d3/a7299b18-4123-434b-8c69-0b9524fffa12/6aed072b-e48f-49d3-9ccf-1a1784592333"
-					(reference "R60")
+					(reference "R78")
 					(unit 1)
 				)
@@
 		(dnp yes)
 		(fields_autoplaced yes)
-		(property "Reference" "R63"
+		(property "Reference" "R73"
 			(at 144.78 46.9899 90)
 			(effects
@@
 			(project "VESA-SBC3399"
 				(path "/ebc9dc57-8b05-484a-a5cd-c53b1efc71d3/a7299b18-4123-434b-8c69-0b9524fffa12/6aed072b-e48f-49d3-9ccf-1a1784592333"
-					(reference "R63")
+					(reference "R73")
 					(unit 1)
 				)
@@
 		(on_board yes)
 		(dnp no)
-		(property "Reference" "#PWR0131"
+		(property "Reference" "#PWR0206"
 			(at 45.72 115.57 0)
 			(effects
@@
 			(project "VESA-SBC3399"
 				(path "/ebc9dc57-8b05-484a-a5cd-c53b1efc71d3/a7299b18-4123-434b-8c69-0b9524fffa12/6aed072b-e48f-49d3-9ccf-1a1784592333"
-					(reference "#PWR0131")
+					(reference "#PWR0206")
 					(unit 1)
 				)
@@
 		(dnp no)
 		(fields_autoplaced yes)
-		(property "Reference" "U1"
+		(property "Reference" "U2"
 			(at 133.35 151.206 0)
 			(effects
@@
 			(project "VESA-SBC3399"
 				(path "/ebc9dc57-8b05-484a-a5cd-c53b1efc71d3/a7299b18-4123-434b-8c69-0b9524fffa12/6aed072b-e48f-49d3-9ccf-1a1784592333"
-					(reference "U1")
+					(reference "U2")
 					(unit 31)
 				)
@@
 		(dnp no)
 		(fields_autoplaced yes)
-		(property "Reference" "U1"
+		(property "Reference" "U2"
 			(at 107.95 45.72 0)
 			(effects
@@
 			(project "VESA-SBC3399"
 				(path "/ebc9dc57-8b05-484a-a5cd-c53b1efc71d3/a7299b18-4123-434b-8c69-0b9524fffa12/6aed072b-e48f-49d3-9ccf-1a1784592333"
-					(reference "U1")
+					(reference "U2")
 					(unit 25)
 				)
@@
 		(on_board yes)
 		(dnp no)
-		(property "Reference" "#PWR0127"
+		(property "Reference" "#PWR0205"
 			(at 78.74 97.79 0)
 			(effects
@@
 			(project "VESA-SBC3399"
 				(path "/ebc9dc57-8b05-484a-a5cd-c53b1efc71d3/a7299b18-4123-434b-8c69-0b9524fffa12/6aed072b-e48f-49d3-9ccf-1a1784592333"
-					(reference "#PWR0127")
+					(reference "#PWR0205")
 					(unit 1)
 				)
@@
 		(dnp no)
 		(fields_autoplaced yes)
-		(property "Reference" "U1"
+		(property "Reference" "U2"
 			(at 224.79 105.495 0)
 			(effects
@@
 			(project "VESA-SBC3399"
 				(path "/ebc9dc57-8b05-484a-a5cd-c53b1efc71d3/a7299b18-4123-434b-8c69-0b9524fffa12/6aed072b-e48f-49d3-9ccf-1a1784592333"
-					(reference "U1")
+					(reference "U2")
 					(unit 30)
 				)
@@
 		(on_board yes)
 		(dnp no)
-		(property "Reference" "#PWR0128"
+		(property "Reference" "#PWR0207"
 			(at 78.74 138.43 0)
 			(effects
@@
 			(project "VESA-SBC3399"
 				(path "/ebc9dc57-8b05-484a-a5cd-c53b1efc71d3/a7299b18-4123-434b-8c69-0b9524fffa12/6aed072b-e48f-49d3-9ccf-1a1784592333"
-					(reference "#PWR0128")
+					(reference "#PWR0207")
 					(unit 1)
 				)
@@
 		(dnp no)
 		(fields_autoplaced yes)
-		(property "Reference" "U1"
+		(property "Reference" "U2"
 			(at 125.73 113.1105 0)
 			(effects
@@
 			(project "VESA-SBC3399"
 				(path "/ebc9dc57-8b05-484a-a5cd-c53b1efc71d3/a7299b18-4123-434b-8c69-0b9524fffa12/6aed072b-e48f-49d3-9ccf-1a1784592333"
-					(reference "U1")
+					(reference "U2")
 					(unit 26)
 				)
@@
 		(on_board yes)
 		(dnp no)
-		(property "Reference" "U1"
+		(property "Reference" "U2"
 			(at 144.78 180.34 0)
 			(effects
@@
 			(project "VESA-SBC3399"
 				(path "/ebc9dc57-8b05-484a-a5cd-c53b1efc71d3/a7299b18-4123-434b-8c69-0b9524fffa12/6aed072b-e48f-49d3-9ccf-1a1784592333"
-					(reference "U1")
+					(reference "U2")
 					(unit 27)
 				)
@@
 		(on_board yes)
 		(dnp no)
-		(property "Reference" "U1"
+		(property "Reference" "U2"
 			(at 196.9456 71.12 0)
 			(effects
@@
 			(project "VESA-SBC3399"
 				(path "/ebc9dc57-8b05-484a-a5cd-c53b1efc71d3/a7299b18-4123-434b-8c69-0b9524fffa12/6aed072b-e48f-49d3-9ccf-1a1784592333"
-					(reference "U1")
+					(reference "U2")
 					(unit 22)
 				)
@@
 		(dnp yes)
 		(fields_autoplaced yes)
-		(property "Reference" "R58"
+		(property "Reference" "R75"
 			(at 81.28 100.3299 90)
 			(effects
@@
 			(project "VESA-SBC3399"
 				(path "/ebc9dc57-8b05-484a-a5cd-c53b1efc71d3/a7299b18-4123-434b-8c69-0b9524fffa12/6aed072b-e48f-49d3-9ccf-1a1784592333"
-					(reference "R58")
+					(reference "R75")
 					(unit 1)
 				)

Commit message: design DDR
Parts:
- renumbered R73 to R144, R74 to R145, R75 to R146, R76 to R147, R77 to R148, R78 to R149, U2 to U17
Connections:
- net GPIO1_A1: now reaches U17.T31 (GPIO1_A1/ISP0_SHUTTER_TRIG/ISP1_SHUTTER_TRIG/TCPD_CC0_VCONN_EN)
- no-connect marks 24 -> 23
Changed lines of the file:
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@@
 	)
 	(no_connect
-		(at 162.56 83.82)
-	)
-	(no_connect
 		(at 220.98 60.96)
 	)
@@
 	(wire
 		(pts
+			(xy 139.7 83.82) (xy 162.56 83.82)
+		)
+		(stroke
+			(width 0)
+			(type default)
+		)
+	)
+	(wire
+		(pts
 			(xy 76.2 187.96) (xy 101.6 187.96)
 		)
@@
 		)
 	)
-	(label "VBUS_USBC0_PWR_EN"
+	(label "VBUS_USBC_PWR_EN"
 		(at 142.24 88.9 0)
 		(effects
@@
 		)
 	)
+	(label "USBC1_INT#"
+		(at 142.24 83.82 0)
+		(effects
+			(font
+				(size 1.27 1.27)
+			)
+			(justify left bottom)
+		)
+	)
 	(label "CPU_I2C4_SDA"
 		(at 55.88 109.22 0)
@@
 		)
 	)
+	(hierarchical_label "GPIO1_A1"
+		(shape input)
+		(at 139.7 83.82 180)
+		(effects
+			(font
+				(size 1.27 1.27)
+			)
+			(justify right)
+		)
+	)
 	(hierarchical_label "I2C4"
 		(shape bidirectional)
@@
 		(dnp no)
 		(fields_autoplaced yes)
-		(property "Reference" "U2"
+		(property "Reference" "U17"
 			(at 248.9182 30.48 0)
 			(effects
@@
 		)
 		(property "Footprint" "footprints:BGA828C65P31X31_2100X2100X161"
-			(at 251.46 55.88 0)
+			(at 248.92 55.88 0)
 			(effects
 				(font
@@
 			(project "VESA-SBC3399"
 				(path "/ebc9dc57-8b05-484a-a5cd-c53b1efc71d3/a7299b18-4123-434b-8c69-0b9524fffa12/6aed072b-e48f-49d3-9ccf-1a1784592333"
-					(reference "U2")
+					(reference "U17")
 					(unit 32)
 				)
@@
 		(dnp yes)
 		(fields_autoplaced yes)
-		(property "Reference" "R74"
-			(at 154.94 46.9899 90)
+		(property "Reference" "R145"
+			(at 160.02 46.9899 90)
 			(effects
 				(font
 					(size 1.27 1.27)
 				)
-				(justify left)
+				(justify right)
 			)
 		)
@@
 		)
 		(property "Resistance" "1kΩ"
-			(at 154.94 49.5299 90)
+			(at 160.02 49.5299 90)
 			(effects
 				(font
 					(size 1.27 1.27)
 				)
-				(justify left)
+				(justify right)
 			)
 		)
 		(property "Tolerance" "±1%"
-			(at 154.94 52.0699 90)
+			(at 160.02 52.0699 90)
 			(effects
 				(font
 					(size 1.27 1.27)
 				)
-				(justify left)
+				(justify right)
 			)
 		)
@@
 			(project "VESA-SBC3399"
 				(path "/ebc9dc57-8b05-484a-a5cd-c53b1efc71d3/a7299b18-4123-434b-8c69-0b9524fffa12/6aed072b-e48f-49d3-9ccf-1a1784592333"
-					(reference "R74")
+					(reference "R145")
 					(unit 1)
 				)
@@
 		(dnp yes)
 		(fields_autoplaced yes)
-		(property "Reference" "R76"
+		(property "Reference" "R147"
 			(at 91.44 100.3299 90)
 			(effects
@@
 			(project "VESA-SBC3399"
 				(path "/ebc9dc57-8b05-484a-a5cd-c53b1efc71d3/a7299b18-4123-434b-8c69-0b9524fffa12/6aed072b-e48f-49d3-9ccf-1a1784592333"
-					(reference "R76")
+					(reference "R147")
 					(unit 1)
 				)
@@
 		(on_board yes)
 		(dnp no)
-		(property "Reference" "#PWR0204"
+		(property "Reference" "#PWR0364"
 			(at 157.48 44.45 0)
 			(effects
@@
 			(project "VESA-SBC3399"
 				(path "/ebc9dc57-8b05-484a-a5cd-c53b1efc71d3/a7299b18-4123-434b-8c69-0b9524fffa12/6aed072b-e48f-49d3-9ccf-1a1784592333"
-					(reference "#PWR0204")
+					(reference "#PWR0364")
 					(unit 1)
 				)
@@
 		(dnp yes)
 		(fields_autoplaced yes)
-		(property "Reference" "R77"
+		(property "Reference" "R148"
 			(at 81.28 140.9699 90)
 			(effects
@@
 			(project "VESA-SBC3399"
 				(path "/ebc9dc57-8b05-484a-a5cd-c53b1efc71d3/a7299b18-4123-434b-8c69-0b9524fffa12/6aed072b-e48f-49d3-9ccf-1a1784592333"
-					(reference "R77")
+					(reference "R148")
 					(unit 1)
 				)
@@
 		(dnp yes)
 		(fields_autoplaced yes)
-		(property "Reference" "R78"
+		(property "Reference" "R149"
 			(at 91.44 140.9699 90)
 			(effects
@@
 			(project "VESA-SBC3399"
 				(path "/ebc9dc57-8b05-484a-a5cd-c53b1efc71d3/a7299b18-4123-434b-8c69-0b9524fffa12/6aed072b-e48f-49d3-9ccf-1a1784592333"
-					(reference "R78")
+					(reference "R149")
 					(unit 1)
 				)
@@
 		(dnp yes)
 		(fields_autoplaced yes)
-		(property "Reference" "R73"
-			(at 144.78 46.9899 90)
+		(property "Reference" "R144"
+			(at 149.86 46.9899 90)
 			(effects
 				(font
 					(size 1.27 1.27)
 				)
-				(justify left)
+				(justify right)
 			)
 		)
@@
 		)
 		(property "Resistance" "1kΩ"
-			(at 144.78 49.5299 90)
+			(at 149.86 49.5299 90)
 			(effects
 				(font
 					(size 1.27 1.27)
 				)
-				(justify left)
+				(justify right)
 			)
 		)
 		(property "Tolerance" "±1%"
-			(at 144.78 52.0699 90)
+			(at 149.86 52.0699 90)
 			(effects
 				(font
 					(size 1.27 1.27)
 				)
-				(justify left)
+				(justify right)
 			)
 		)
@@
 			(project "VESA-SBC3399"
 				(path "/ebc9dc57-8b05-484a-a5cd-c53b1efc71d3/a7299b18-4123-434b-8c69-0b9524fffa12/6aed072b-e48f-49d3-9ccf-1a1784592333"
-					(reference "R73")
+					(reference "R144")
 					(unit 1)
 				)
@@
 		(on_board yes)
 		(dnp no)
-		(property "Reference" "#PWR0206"
+		(property "Reference" "#PWR0366"
 			(at 45.72 115.57 0)
 			(effects
@@
 			(project "VESA-SBC3399"
 				(path "/ebc9dc57-8b05-484a-a5cd-c53b1efc71d3/a7299b18-4123-434b-8c69-0b9524fffa12/6aed072b-e48f-49d3-9ccf-1a1784592333"
-					(reference "#PWR0206")
+					(reference "#PWR0366")
 					(unit 1)
 				)
@@
 		(dnp no)
 		(fields_autoplaced yes)
-		(property "Reference" "U2"
+		(property "Reference" "U17"
 			(at 133.35 151.206 0)
 			(effects
@@
 			(project "VESA-SBC3399"
 				(path "/ebc9dc57-8b05-484a-a5cd-c53b1efc71d3/a7299b18-4123-434b-8c69-0b9524fffa12/6aed072b-e48f-49d3-9ccf-1a1784592333"
-					(reference "U2")
+					(reference "U17")
 					(unit 31)
 				)
@@
 		(dnp no)
 		(fields_autoplaced yes)
-		(property "Reference" "U2"
+		(property "Reference" "U17"
 			(at 107.95 45.72 0)
 			(effects
@@
 		)
 		(property "Footprint" "footprints:BGA828C65P31X31_2100X2100X161"
-			(at 109.22 66.04 0)
+			(at 106.68 66.04 0)
 			(effects
 				(font
@@
 			(project "VESA-SBC3399"
 				(path "/ebc9dc57-8b05-484a-a5cd-c53b1efc71d3/a7299b18-4123-434b-8c69-0b9524fffa12/6aed072b-e48f-49d3-9ccf-1a1784592333"
-					(reference "U2")
+					(reference "U17")
 					(unit 25)
 				)
@@
 		(on_board yes)
 		(dnp no)
-		(property "Reference" "#PWR0205"
+		(property "Reference" "#PWR0365"
 			(at 78.74 97.79 0)
 			(effects
@@
 			(project "VESA-SBC3399"
 				(path "/ebc9dc57-8b05-484a-a5cd-c53b1efc71d3/a7299b18-4123-434b-8c69-0b9524fffa12/6aed072b-e48f-49d3-9ccf-1a1784592333"
-					(reference "#PWR0205")
+					(reference "#PWR0365")
 					(unit 1)
 				)
@@
 		(dnp no)
 		(fields_autoplaced yes)
-		(property "Reference" "U2"
+		(property "Reference" "U17"
 			(at 224.79 105.495 0)
 			(effects
@@
 			(project "VESA-SBC3399"
 				(path "/ebc9dc57-8b05-484a-a5cd-c53b1efc71d3/a7299b18-4123-434b-8c69-0b9524fffa12/6aed072b-e48f-49d3-9ccf-1a1784592333"
-					(reference "U2")
+					(reference "U17")
 					(unit 30)
 				)
@@
 		(on_board yes)
 		(dnp no)
-		(property "Reference" "#PWR0207"
+		(property "Reference" "#PWR0367"
 			(at 78.74 138.43 0)
 			(effects
@@
 			(project "VESA-SBC3399"
 				(path "/ebc9dc57-8b05-484a-a5cd-c53b1efc71d3/a7299b18-4123-434b-8c69-0b9524fffa12/6aed072b-e48f-49d3-9ccf-1a1784592333"
-					(reference "#PWR0207")
+					(reference "#PWR0367")
 					(unit 1)
 				)
@@
 		(dnp no)
 		(fields_autoplaced yes)
-		(property "Reference" "U2"
+		(property "Reference" "U17"
 			(at 125.73 113.1105 0)
 			(effects
@@
 			(project "VESA-SBC3399"
 				(path "/ebc9dc57-8b05-484a-a5cd-c53b1efc71d3/a7299b18-4123-434b-8c69-0b9524fffa12/6aed072b-e48f-49d3-9ccf-1a1784592333"
-					(reference "U2")
+					(reference "U17")
 					(unit 26)
 				)
@@
 		(on_board yes)
 		(dnp no)
-		(property "Reference" "U2"
+		(property "Reference" "U17"
 			(at 144.78 180.34 0)
 			(effects
@@
 		)
 		(property "Footprint" "footprints:BGA828C65P31X31_2100X2100X161"
-			(at 142.24 187.96 0)
+			(at 124.46 187.96 0)
 			(effects
 				(font
@@
 			(project "VESA-SBC3399"
 				(path "/ebc9dc57-8b05-484a-a5cd-c53b1efc71d3/a7299b18-4123-434b-8c69-0b9524fffa12/6aed072b-e48f-49d3-9ccf-1a1784592333"
-					(reference "U2")
+					(reference "U17")
 					(unit 27)
 				)
@@
 		(on_board yes)
 		(dnp no)
-		(property "Reference" "U2"
+		(property "Reference" "U17"
 			(at 196.9456 71.12 0)
 			(effects
@@
 			(project "VESA-SBC3399"
 				(path "/ebc9dc57-8b05-484a-a5cd-c53b1efc71d3/a7299b18-4123-434b-8c69-0b9524fffa12/6aed072b-e48f-49d3-9ccf-1a1784592333"
-					(reference "U2")
+					(reference "U17")
 					(unit 22)
 				)
@@
 		(dnp yes)
 		(fields_autoplaced yes)
-		(property "Reference" "R75"
+		(property "Reference" "R146"
 			(at 81.28 100.3299 90)
 			(effects
@@
 			(project "VESA-SBC3399"
 				(path "/ebc9dc57-8b05-484a-a5cd-c53b1efc71d3/a7299b18-4123-434b-8c69-0b9524fffa12/6aed072b-e48f-49d3-9ccf-1a1784592333"
-					(reference "R75")
+					(reference "R146")
 					(unit 1)
 				)
