File: CPU-RK3399_SDIO.kicad_sch (KiCad schematic)
At the start: 7 parts, among them U1 RK3399

Commit message: update design power
Parts:
- renumbered R51 to R24, R52 to R25, R53 to R26, R54 to R27, R55 to R28, R56 to R29, U1 to U2
Changed lines of the file:
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@@
 		(on_board yes)
 		(dnp no)
-		(property "Reference" "R55"
+		(property "Reference" "R28"
 			(at 114.3 92.71 0)
 			(effects
@@
 			(project "VESA-SBC3399"
 				(path "/ebc9dc57-8b05-484a-a5cd-c53b1efc71d3/a7299b18-4123-434b-8c69-0b9524fffa12/72ea5c00-7e69-4de6-bdd7-dbdcea913c16"
-					(reference "R55")
+					(reference "R28")
 					(unit 1)
 				)
@@
 		(on_board yes)
 		(dnp no)
-		(property "Reference" "R53"
+		(property "Reference" "R26"
 			(at 114.3 87.63 0)
 			(effects
@@
 			(project "VESA-SBC3399"
 				(path "/ebc9dc57-8b05-484a-a5cd-c53b1efc71d3/a7299b18-4123-434b-8c69-0b9524fffa12/72ea5c00-7e69-4de6-bdd7-dbdcea913c16"
-					(reference "R53")
+					(reference "R26")
 					(unit 1)
 				)
@@
 		(on_board yes)
 		(dnp no)
-		(property "Reference" "R51"
+		(property "Reference" "R24"
 			(at 114.3 82.55 0)
 			(effects
@@
 			(project "VESA-SBC3399"
 				(path "/ebc9dc57-8b05-484a-a5cd-c53b1efc71d3/a7299b18-4123-434b-8c69-0b9524fffa12/72ea5c00-7e69-4de6-bdd7-dbdcea913c16"
-					(reference "R51")
+					(reference "R24")
 					(unit 1)
 				)
@@
 		(on_board yes)
 		(dnp no)
-		(property "Reference" "R52"
+		(property "Reference" "R25"
 			(at 114.3 85.09 0)
 			(effects
@@
 			(project "VESA-SBC3399"
 				(path "/ebc9dc57-8b05-484a-a5cd-c53b1efc71d3/a7299b18-4123-434b-8c69-0b9524fffa12/72ea5c00-7e69-4de6-bdd7-dbdcea913c16"
-					(reference "R52")
+					(reference "R25")
 					(unit 1)
 				)
@@
 		(on_board yes)
 		(dnp no)
-		(property "Reference" "R56"
+		(property "Reference" "R29"
 			(at 114.3 95.25 0)
 			(effects
@@
 			(project "VESA-SBC3399"
 				(path "/ebc9dc57-8b05-484a-a5cd-c53b1efc71d3/a7299b18-4123-434b-8c69-0b9524fffa12/72ea5c00-7e69-4de6-bdd7-dbdcea913c16"
-					(reference "R56")
+					(reference "R29")
 					(unit 1)
 				)
@@
 		(dnp no)
 		(fields_autoplaced yes)
-		(property "Reference" "U1"
+		(property "Reference" "U2"
 			(at 149.8451 73.66 0)
 			(effects
@@
 			(project "VESA-SBC3399"
 				(path "/ebc9dc57-8b05-484a-a5cd-c53b1efc71d3/a7299b18-4123-434b-8c69-0b9524fffa12/72ea5c00-7e69-4de6-bdd7-dbdcea913c16"
-					(reference "U1")
+					(reference "U2")
 					(unit 13)
 				)
@@
 		(on_board yes)
 		(dnp no)
-		(property "Reference" "R54"
+		(property "Reference" "R27"
 			(at 114.3 90.17 0)
 			(effects
@@
 			(project "VESA-SBC3399"
 				(path "/ebc9dc57-8b05-484a-a5cd-c53b1efc71d3/a7299b18-4123-434b-8c69-0b9524fffa12/72ea5c00-7e69-4de6-bdd7-dbdcea913c16"
-					(reference "R54")
+					(reference "R27")
 					(unit 1)
 				)

Commit message: design DDR
Parts:
- renumbered R29 to R100, R24 to R95, R25 to R96, R26 to R97, R27 to R98, R28 to R99, U2 to U17
Changed lines of the file:
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@@
 		(on_board yes)
 		(dnp no)
-		(property "Reference" "R28"
+		(property "Reference" "R99"
 			(at 114.3 92.71 0)
 			(effects
@@
 			(project "VESA-SBC3399"
 				(path "/ebc9dc57-8b05-484a-a5cd-c53b1efc71d3/a7299b18-4123-434b-8c69-0b9524fffa12/72ea5c00-7e69-4de6-bdd7-dbdcea913c16"
-					(reference "R28")
+					(reference "R99")
 					(unit 1)
 				)
@@
 		(on_board yes)
 		(dnp no)
-		(property "Reference" "R26"
+		(property "Reference" "R97"
 			(at 114.3 87.63 0)
 			(effects
@@
 			(project "VESA-SBC3399"
 				(path "/ebc9dc57-8b05-484a-a5cd-c53b1efc71d3/a7299b18-4123-434b-8c69-0b9524fffa12/72ea5c00-7e69-4de6-bdd7-dbdcea913c16"
-					(reference "R26")
+					(reference "R97")
 					(unit 1)
 				)
@@
 		(on_board yes)
 		(dnp no)
-		(property "Reference" "R24"
+		(property "Reference" "R95"
 			(at 114.3 82.55 0)
 			(effects
@@
 			(project "VESA-SBC3399"
 				(path "/ebc9dc57-8b05-484a-a5cd-c53b1efc71d3/a7299b18-4123-434b-8c69-0b9524fffa12/72ea5c00-7e69-4de6-bdd7-dbdcea913c16"
-					(reference "R24")
+					(reference "R95")
 					(unit 1)
 				)
@@
 		(on_board yes)
 		(dnp no)
-		(property "Reference" "R25"
+		(property "Reference" "R96"
 			(at 114.3 85.09 0)
 			(effects
@@
 			(project "VESA-SBC3399"
 				(path "/ebc9dc57-8b05-484a-a5cd-c53b1efc71d3/a7299b18-4123-434b-8c69-0b9524fffa12/72ea5c00-7e69-4de6-bdd7-dbdcea913c16"
-					(reference "R25")
+					(reference "R96")
 					(unit 1)
 				)
@@
 		(on_board yes)
 		(dnp no)
-		(property "Reference" "R29"
+		(property "Reference" "R100"
 			(at 114.3 95.25 0)
 			(effects
@@
 			(project "VESA-SBC3399"
 				(path "/ebc9dc57-8b05-484a-a5cd-c53b1efc71d3/a7299b18-4123-434b-8c69-0b9524fffa12/72ea5c00-7e69-4de6-bdd7-dbdcea913c16"
-					(reference "R29")
+					(reference "R100")
 					(unit 1)
 				)
@@
 		(dnp no)
 		(fields_autoplaced yes)
-		(property "Reference" "U2"
+		(property "Reference" "U17"
 			(at 149.8451 73.66 0)
 			(effects
@@
 		)
 		(property "Footprint" "footprints:BGA828C65P31X31_2100X2100X161"
-			(at 167.64 96.52 0)
+			(at 149.86 96.52 0)
 			(effects
 				(font
@@
 			(project "VESA-SBC3399"
 				(path "/ebc9dc57-8b05-484a-a5cd-c53b1efc71d3/a7299b18-4123-434b-8c69-0b9524fffa12/72ea5c00-7e69-4de6-bdd7-dbdcea913c16"
-					(reference "U2")
+					(reference "U17")
 					(unit 13)
 				)
@@
 		(on_board yes)
 		(dnp no)
-		(property "Reference" "R27"
+		(property "Reference" "R98"
 			(at 114.3 90.17 0)
 			(effects
@@
 			(project "VESA-SBC3399"
 				(path "/ebc9dc57-8b05-484a-a5cd-c53b1efc71d3/a7299b18-4123-434b-8c69-0b9524fffa12/72ea5c00-7e69-4de6-bdd7-dbdcea913c16"
-					(reference "R27")
+					(reference "R98")
 					(unit 1)
 				)
