File: CPU-RK3399_USB.kicad_sch (KiCad schematic)
At the start: 18 parts, among them U1 RK3399

Commit message: update design power
Parts:
- renumbered C92 to C147, C93 to C148, C94 to C149, C95 to C150, C96 to C151, C97 to C152, C98 to C153, C99 to C154, C100 to C155, R19 to R42, R20 to R43, R21 to R44, R22 to R45, R23 to R46, R24 to R47, TP3 to TP4, TP4 to TP5, U1 to U2

Commit message: design DDR
Parts:
- R117: renamed from R46; footprint footprints: -> footprints:RESC1608X45N
- R118: renamed from R47; footprint footprints: -> footprints:RESC1608X45N
- renumbered C147 to C274, C148 to C275, C149 to C276, C150 to C277, C151 to C278, C152 to C279, C153 to C280, C154 to C281, C155 to C282, R42 to R113, R43 to R114, R44 to R115, R45 to R116, U2 to U17
Connections:
- net TYPEC0_U2VBUSDET: now reaches U17.AK30 (TYPEC0_U2VBUSDET)
- net TYPEC1_U2VBUSDET: now reaches U17.AK31 (TYPEC1_U2VBUSDET)
Other:
- moved on the sheet: C280, C281, C282, R113, R114, R115, R116, R117, R118, U17O
