File: Power.kicad_sch (KiCad schematic)
At the start: 0 parts

Commit message: design CPU-RK3399 eMMC Controller
Other:
- company: (none) -> TickLab
Changed lines of the file:
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@@
 	(paper "A4")
 	(title_block
-		(date "2026-01-09")
+		(date "2026-01-14")
 		(rev "1.0.0")
+		(company "TickLab")
 	)
 )

Commit message: design PMIC
Other:
- added sheet Power DC-IN (Power_DC-IN.kicad_sch)
- added sheet Power PMIC (Power_PMIC.kicad_sch)
- title: (none) -> Power

Commit message: update design power
Parts:
- added BAT1: ~, footprints:, symbol component_library:Connectors/CR1220-2
- added BTN1, BTN2: ~, footprints:, symbol component_library:Switches, Buttons/TSA016A2518A
- added C1, C12, C2: ~, footprints:CAPC1005X50N, symbol component_library:Capacitors/CL05A106MQ5NUNC
- added C10: ~, footprints:CAPC1005X50N, symbol component_library:Capacitors/0402CG470J500NT
- added C11, C16, C166, C175, C186, C200, C215, C226, C5, C6: ~, footprints:CAPC1005X50N, symbol component_library:Capacitors/0402CG180J500NT
- added C13, C14, C15, C168, C169, C170, C171, C177, C178, C179, C180, C183, C184, C185, C3, C4, C7: ~, footprints:CAPC1608X80N, symbol component_library:Capacitors/CL10A226MQ8NRNC
- added C164, C173, C189, C191, C224, C42: ~, footprints:CAPC1608X80N, symbol component_library:Capacitors/CL10A106MA8NRNC
- added C165, C167, C17, C172, C174, C176, C181, C187, C188, C19, C190, C27, C33, C37, C41, C44, C45: ~, footprints:CAPC1005X50N, symbol component_library:Capacitors/CL05B104KO5NNNC
- added C18, C20, C202, C211, C212, C213, C217, C228, C23, C230, C26, C28, C30, C32, C34, C36, C38: ~, footprints:CAPC1005X50N, symbol component_library:Capacitors/CL05A105KA5NQNC
- added C182, C199, C201, C207, C214, C216, C222, C225, C227: ~, footprints:CAPC1005X50N, symbol component_library:Capacitors/CL05B104KB54PNC
- added C198: ~, footprints:, symbol component_library:Capacitors/CL21B105KBFNNNE
- added C203, C204, C223, C229: ~, footprints:, symbol component_library:Capacitors/CL21A226MAQNNNE
- added C205: ~, footprints:CAPC1005X50N, symbol component_library:Capacitors/0402B472K500NT
- added C206: ~, footprints:, symbol component_library:Capacitors/0603B222K500NT
- added C208, C209, C210: ~, footprints:, symbol component_library:Capacitors/CL21A475KAQNNNE
- added C21, C24, C25, C31, C35: ~, footprints:CAPC1608X80N, symbol component_library:Capacitors/CL10A225KO8NNNC
- added C218, C219: ~, footprints:, symbol component_library:Capacitors/CL21A476MQYNNNE
- added C22, C29: ~, footprints:CAPC1005X50N, symbol component_library:Capacitors/CL05A475MP5NRNC
- added C220: ~, footprints:CAPC1005X50N, symbol component_library:Capacitors/CC0402KRX5R6BB124
- added C221, C46: ~, footprints:CAPC1005X50N, symbol component_library:Capacitors/CL05A225MQ5NSNC
- added C231: ~, footprints:CAPC1005X50N, symbol component_library:Capacitors/0402B223K500NT
- added C39, C40: ~, footprints:CAPC1005X50N, symbol component_library:Capacitors/0402CG220J500NT
- added C43: ~, footprints:CAPC1005X50N, symbol component_library:Capacitors/0402B102K500NT
- added C8, C9: ~, footprints:CAPC2012X115N, symbol component_library:Capacitors/CL21A226MAQNNNE
- added CON2: ~, footprints:, symbol component_library:Connectors/DC-091
- added D1: ~, footprints:, symbol component_library:TVS, ESD/AZ5825-01F
- added D10, D11: ~, footprints:, symbol component_library:TVS, ESD/SMAJ12A
- added D2: ~, footprints:, symbol component_library:Diodes/BAT54C
- added D3, D4, D5: ~, footprints:, symbol component_library:Diodes/B5819WS
- added D6: ~, footprints:, symbol component_library:TVS, ESD/ESD5Z2.5T1G
- added L1: ~, footprints:CRH201610S-1R0MT, symbol component_library:Inductors/CRH201610S-1R0MT
- added L2: ~, footprints:VLS201610CX-2R2M-1, symbol component_library:Inductors/VLS201610CX-2R2M-1
- added L3, L9: ~, footprints:FXLB252012-2R2-M, symbol component_library:Inductors/FXLB252012-2R2-M
- added L4: ~, footprints:NRSE2512-1R0M, symbol component_library:Inductors/NRSE2512-1R0M
- added L5, L6: ~, footprints:WIP201610P-R24ML, symbol component_library:Inductors/WIP201610P-R24ML
- added L7: ~, footprints:, symbol component_library:Inductors/IHLP2525EZER1R0M01
- added L8: ~, footprints:ETQP3M1R5KVP, symbol component_library:Inductors/ETQP3M1R5KVP
- added Q1: ~, footprints:, symbol component_library:FETs/WPM2341-3/TR
- added Q2: ~, footprints:, symbol component_library:BJTs/S8050
- added R1, R2, R4, R79, R81: ~, footprints:RESC1005X35N, symbol component_library:Resistors/0402WGF1000TCE
- added R10: ~, footprints:RESC1608X45N, symbol component_library:Resistors/0603WAF1503T5E
- added R102: ~, footprints:RESC1608X45N, symbol component_library:Resistors/0603WAF4703T5E
- added R103, R108, R109, R14: ~, footprints:RESC1005X35N, symbol component_library:Resistors/0402WGF4702TCE
- added R104: ~, footprints:RESC1608X45N, symbol component_library:Resistors/0603WAF2702T5E
- added R105, R107, R115, R116, R13, R7, R8, R80, R82, R84, R9: ~, footprints:RESC1005X35N, symbol component_library:Resistors/0402WGF1002TCE
- added R106: ~, footprints:RESC1608X45N, symbol component_library:Resistors/0603WAF5601T5E
- added R11: ~, footprints:RESC1005X35N, symbol component_library:Resistors/0402WGF2703TCE
- added R110: ~, footprints:RESC1608X45N, symbol component_library:Resistors/0603WAF8200T5E
- added R111, R112: ~, footprints:RESC1005X35N, symbol component_library:Resistors/0402WGF0000TCE
- added R113: ~, footprints:RESC1608X45N, symbol component_library:Resistors/0603WAF8202T5E
- added R114: ~, footprints:, symbol component_library:Resistors/0805W8F7322T5E
- added R117, R119: ~, footprints:RESC1005X35N, symbol component_library:Resistors/0402WGF3012TCE
- added R118: ~, footprints:RESC1005X35N, symbol component_library:Resistors/0402WGF4871TCE
- added R12, R124: ~, footprints:RESC1005X35N, symbol component_library:Resistors/0402WGF1003TCE
- added R120, R122, R123: ~, footprints:RESC1005X35N, symbol component_library:Resistors/0402WGF2002TCE
- added R121: ~, footprints:RESC1005X35N, symbol component_library:Resistors/0402WGF1473TCE
- added R3: ~, footprints:RESC1608X45N, symbol component_library:Resistors/0603WAF1203T5E
- added R5: ~, footprints:RESC1005X35N, symbol component_library:Resistors/0402WGF4302TCE
- added R6: ~, footprints:, symbol component_library:Resistors/1206W4F100LT5E
- added R83: ~, footprints:RESC1005X35N, symbol component_library:Resistors/0402WGF3322TCE
- added R86: ~, footprints:RESC1005X35N, symbol component_library:Resistors/0402WGF2403TCE
- added U1: RK808-D, footprints:, symbol component_library:PMIC/RK808-D
- added U3: SYR837PKC, footprints:, symbol component_library:PMIC/SYR837PKC
- added U4: SYR838PKC, footprints:, symbol component_library:PMIC/SYR838PKC
- added U5: TPS563201DDCR, footprints:, symbol component_library:PMIC/TPS563201DDCR
- added U6: TPS25974ARPWR, footprints:, symbol component_library:PMIC/TPS25974ARPWR
- added U7: TPS548A28RWWR, footprints:, symbol component_library:PMIC/TPS548A28RWWR
- added U8: TPS51386RJNR, symbol component_library_symbols:TPS51386RJNR
- added Y1: ~, footprints:, symbol component_library:Crystals, Oscillators, Resonators/Q13FC13500004
Connections:
- net PMIC_CLK32KOUT1: now also R7.2, U1.68 (CLK32KOUT1)
- net PMIC_CLK32KOUT2: now also U1.67 (CLK32KOUT2)
- net PMIC_INT: now also U1.49 (INT)
- net PMIC_NRESPWRON: now also C41.1, R8.2, U1.20 (NRESPWRON)
- net PMIC_OTP: now also D5.A (Anode)
- net PMIC_PWRON: now also BTN2.3, BTN2.4, C45.1, D4.A (Anode), D4.C (Cathode), D6.C (Cathode), R9.2, U1.51 (PWRON)
- net PMIC_SLEEP: now also U1.50 (SLEEP)
- new net: C182.1, U5.6 (VBST)
- new net: C19.1, U1.31 (VLDO1)
- new net: C32.1, U1.8 (VCC8)
- new net: C221.1, R119.2, U7.19 (VCC)
- new net: C222.1, U8.8 (VBST)
- new net: C230.1, R124.1, U8.9 (VCC)
- new net: C43.1, R10.1, R11.1, U1.34 (VDC)
- new net: C42.2, D3.C (Cathode), R10.2
- new net: D2.3 (Cathode), R6.2
- new net: Q2.B (Base), R13.1, R14.1
- new net: Q1.G (Gate), Q2.C (Collector), R12.2
- new net: C207.1, U7.1 (BOOT)
- new net: R119.1, U7.9 (PGOOD)
- new net: C46.1, D5.C (Cathode), R13.2
- new net: C33.1, U1.7 (VSWOUT1)
- new net: R124.2, U8.3 (PG)
- new net: C231.1, U8.5 (SS)
- new net: C17.1, U1.37 (VREF)
- new net: R2.2, R5.2
- new net: R104.2, R107.1, R108.1
- new net: C27.1, U1.14 (VLDO5)
- new net +0V9_AVCC_HDMI: C24.1, U1.5 (VLDO7)
- new net +0V9_VDD_CENTER: C3.1, C4.1, C5.1, L1.1, R1.1
- new net +0V9_VDD_CPU_B: C166.1, C167.1, C168.1, C169.1, C170.1, C171.1, L5.2, R79.2
- new net +0V9_VDD_CPU_L: C14.1, C15.1, C16.1, L4.1, R4.1
- new net +0V9_VDD_GPU: C175.1, C176.1, C177.1, C178.1, C179.1, C180.1, L6.2, R81.2
- new net +12V_DC_IN: C198.1, C199.1, CON2.P, D10.C (Cathode), R102.1, U6.5 (IN)
- new net +12V_SYS: C200.1, C201.1, C202.1, C203.1, C204.1, C208.1, C209.1, C210.1, C211.1, C212.1, C213.1, C214.1, C223.1, C224.1, C225.1, D11.C (Cathode), R103.1, R104.1, R113.1, R120.1, U6.6 (OUT), U7.10 (VIN), U7.21 (VIN), U8.1 (VIN)
- new net +1V35_VCC_DDR: C10.1, C11.1, C12.1, C13.1, L3.2, R2.1
- new net +1V5_VCC: C29.1, U1.2 (VLDO6)
- new net +1V8_AVCC: C22.1, U1.3 (VLDO3)
- new net +1V8_AVCC_HDMI: C21.1, U1.33 (VLDO2)
- new net +1V8_VCC: C38.1, C6.1, C7.1, L2.2, R7.1, R8.1, R80.1, R82.1, U1.17 (VDDIO), U1.63 (VFB4)
- new net +3V0_IOVCC_SD: C25.1, U1.12 (VLDO4)
- new net +3V0_VCC: C31.1, U1.15 (VLDO8)
- new net +3V0_VCC_BAT: BAT1.P, D2.2 (Anode)
- new net +3V0_VCC_RTC: BTN1.1, BTN1.2, C36.1, C37.1, Q1.S (Source), R12.1, R6.1, R9.1, U1.52 (BOOT0), U1.53 (BOOT1), U1.9 (VCCRTC)
- new net +3V0_VCC_S0: C35.1, U1.11 (VSWOUT2)
- new net +3V3_VCC_SYS: C183.1, C184.1, C185.1, C186.1, C187.1, C34.1, L9.2, R83.1, U1.10 (VCC12)
- new net +5V0_SYS: C1.1, C164.1, C165.1, C173.1, C174.1, C18.1, C189.1, C190.1, C191.1, C2.1, C20.1, C226.1, C227.1, C228.1, C229.1, C23.1, C26.1, C28.1, C30.1, C42.1, C8.1, C9.1, D1.1, D2.1 (Anode), L8.2, R121.1, U1.1 (VCC10), U1.13 (VCC9), U1.16 (VCC11), U1.23 (VCC2_1), U1.24 (VCC2_2), U1.32 (VCC6), U1.35 (VLDOA), U1.36 (VCCA), U1.4 (VCC7), U1.44 (VCC1_1), U1.45 (VCC1_2), U1.59 (VCC3), U1.60 (VCC4), U3.D1 (VIN), U3.D2 (VIN), U3.E1 (VIN), U3.E2 (VIN), U4.D1 (VIN), U4.D2 (VIN), U4.E1 (VIN), U4.E2 (VIN), U5.3 (VIN)
- new net +5V0_USB: C215.1, C216.1, C217.1, C218.1, C219.1, L7.2, R114.1
- new net +5V0_VPP_OTP: BTN1.3, BTN1.4, C44.1, Q1.D (Drain), U1.6 (VPPOTP)
- new net 0V9_VDD_CENTER_FB: R1.2, U1.39 (VFB1)
- new net 0V9_VDD_CENTER_SW: L1.2, U1.42 (SW1_1), U1.43 (SW1_2)
- new net 0V9_VDD_CPU_B_FB: R79.1, U3.A4 (VOUT)
- new net 0V9_VDD_CPU_B_PWR_EN: C172.1, R80.2, U3.A2 (EN)
- new net 0V9_VDD_CPU_B_SW: L5.1, U3.D3 (SW), U3.D4 (SW), U3.E3 (SW), U3.E4 (SW)
- new net 0V9_VDD_CPU_B_VSEL: U3.A1 (VSEL)
- new net 0V9_VDD_CPU_L_FB: R4.2, U1.29 (VFB2)
- new net 0V9_VDD_CPU_L_SW: L4.2, U1.25 (SW2_1), U1.26 (SW2_2)
- new net 0V9_VDD_GPU_FB: R81.1, U4.A4 (VOUT)
- new net 0V9_VDD_GPU_PWR_EN: C181.1, R82.2, U4.A2 (EN)
- new net 0V9_VDD_GPU_SW: L6.1, U4.D3 (SW), U4.D4 (SW), U4.E3 (SW), U4.E4 (SW)
- new net 0V9_VDD_GPU_VSEL: U4.A1 (VSEL)
- new net 12V_SYS_ILM: R110.1, U6.9 (ILM)
- new net 12V_SYS_ITIMER: C206.1, U6.10 (ITIMER)
- new net 12V_SYS_OVLO: R105.2, R109.1, U6.2 (OVLO)
- new net 12V_SYS_PG: R108.2, R111.1, R112.1, U6.3 (PG)
- new net 12V_SYS_PGTH: R103.2, R106.1, U6.4 (PGTH)
- new net 12V_SYS_UVLO: R102.2, R105.1, U6.1 (EN/UVLO)
- new net 12V_SYS_dVdT: C205.1, U6.7 (dV/dT)
- new net 1V35_VCC_DDR_FB: C10.2, R3.1, R5.1, U1.56 (VFB3)
- new net 1V35_VCC_DDR_SW: L3.1, U1.58 (SW3)
- new net 1V8_VCC_SW: L2.1, U1.61 (SW4)
- new net 3V3_VCC_SYS_FB: R83.2, R84.1, U5.4 (VFB)
- new net 3V3_VCC_SYS_PWR_EN: C188.1, R86.2, U5.5 (EN)
- new net 3V3_VCC_SYS_SW: C182.2, L9.1, U5.2 (SW)
- new net 5V0_SYS_FB: R121.2, R123.1, U8.4 (FB)
- new net 5V0_SYS_PWR_EN: R112.2, R120.2, R122.1, U8.11 (EN)
- new net 5V0_SYS_SW: C222.2, L8.1, U8.7 (SW)
- new net 5V0_USB_FB: R114.2, R116.1, U7.7 (FB)
- new net 5V0_USB_MODE: R117.1, U7.4 (MODE)
- new net 5V0_USB_PWR_EN: R111.2, R113.2, R115.1, U7.8 (EN)
- new net 5V0_USB_SS: C220.1, U7.5 (SS/REFIN)
- new net 5V0_USB_SW: C207.2, L7.1, U7.20 (SW)
- new net 5V0_USB_TRIP: R118.1, U7.3 (TRIP)
- new net CPU_I2C0_SCL: U1.19 (SCL), U3.A3 (SCL), U4.A3 (SCL)
- new net CPU_I2C0_SDA: U1.18 (SDA), U3.B1 (SDA), U4.B1 (SDA)
- new net GND: BAT1.N, BTN2.1, BTN2.2, C1.2, C11.2, C12.2, C13.2, C14.2, C15.2, C16.2, C164.2, C165.2, C166.2, C167.2, C168.2, C169.2, C17.2, C170.2, C171.2, C172.2, C173.2, C174.2, C175.2, C176.2, C177.2, C178.2, C179.2, C18.2, C180.2, C181.2, C183.2, C184.2, C185.2, C186.2, C187.2, C188.2, C189.2, C19.2, C190.2, C191.2, C198.2, C199.2, C2.2, C20.2, C200.2, C201.2, C202.2, C203.2, C204.2, C205.2, C206.2, C208.2, C209.2, C21.2, C210.2, C211.2, C212.2, C213.2, C214.2, C215.2, C216.2, C217.2, C218.2, C219.2, C22.2, C220.2, C221.2, C223.2, C224.2, C225.2, C226.2, C227.2, C228.2, C229.2, C23.2, C230.2, C231.2, C24.2, C25.2, C26.2, C27.2, C28.2, C29.2, C3.2, C30.2, C31.2, C32.2, C33.2, C34.2, C35.2, C36.2, C37.2, C38.2, C39.2, C4.2, C40.2, C41.2, C43.2, C44.2, C45.2, C46.2, C5.2, C6.2, C7.2, C8.2, C9.2, CON2.N, D1.2, D10.A (Anode), D11.A (Anode), D3.A (Anode), D6.A (Anode), Q2.E (Emitter), R106.2, R107.2, R109.2, R11.2, R110.2, R115.2, R116.2, R117.2, R118.2, R122.2, R123.2, R14.2, R3.2, R84.2, U1.21 (DVS2), U1.22 (DVS1), U1.27 (GND2_1), U1.28 (GND2_2), U1.30 (AGND), U1.38 (DGND), U1.40 (GND1_1), U1.41 (GND1_2), U1.46 (GND5), U1.57 (GND3), U1.62 (GND4), U1.64 (VREFGND), U1.69 (GND_PAD), U3.B2 (GND), U3.B3 (GND), U3.B4 (AGND), U3.C1 (GND), U3.C2 (GND), U3.C3 (GND), U3.C4 (GND), U4.B2 (GND), U4.B3 (GND), U4.B4 (AGND), U4.C1 (GND), U4.C2 (GND), U4.C3 (GND), U4.C4 (GND), U5.1 (GND), U6.8 (GND), U7.11 (PGND), U7.12 (PGND), U7.13 (PGND), U7.14 (PGND), U7.15 (PGND), U7.16 (PGND), U7.17 (PGND), U7.18 (PGND), U7.2 (AGND), U7.6 (VSNS-), U8.10 (AGND), U8.12 (MODE), U8.2 (PGND)
- new net PMIC_EXT_PWR_EN: R86.1, U1.55 (EXT_EN)
- new net PMIC_OSC32KIN: C39.1, U1.65 (OSC32KIN), Y1.1
- new net PMIC_OSC32KOUT: C40.1, U1.66 (OSC32KOUT), Y1.2 (1)
- no-connect marks 0 -> 1
Other:
- removed sheet Power DC-IN
- removed sheet Power PMIC
- note added: "DC-IN"
- note added: "DDR3: 1.5V DDR3L: 1.35V LPDDR3: 1.25V LPDDR4: 1.13V"
- note added: "PMIC RK808-D"
- note added: "Power of +0V9_VDD_CPU_B"
- note added: "Power of +0V9_VDD_GPU"
- note added: "Power of +3V3_VCC_SYS"
- note added: "Trace > 1.5A"
- note added: "Trace > 1A"
- note added: "Trace > 2.18A"
- note added: "Trace > 2A"
- note added: "Trace > 3.17A"
- note added: "Trace > 3A"
- note added: "Trace > 4.5A"
- note added: "Trace > 5.24A"
- note added: "Trace > 5.35A"
- note added: "Trace > 7.6A"

Commit message: finish design power
Parts:
- added C192, C193, C197, C235: ~, footprints:CAPC1005X50N, symbol component_library:Capacitors/CL05A105KA5NQNC
- added C194, C233, C236: ~, footprints:CAPC1005X50N, symbol component_library:Capacitors/0402CG180J500NT
- added C195, C196, C232, C234, C237, C242, C243: ~, footprints:CAPC1005X50N, symbol component_library:Capacitors/CL05B104KO5NNNC
- added C238: ~, footprints:CAPC1608X80N, symbol component_library:Capacitors/CL10A226MQ8NRNC
- added C239: ~, footprints:CAPC1005X50N, symbol component_library:Capacitors/0402CG470J500NT
- added C240: ~, footprints:CAPC1005X50N, symbol component_library:Capacitors/0402B223K500NT
- added C241: ~, footprints:CAPC1608X80N, symbol component_library:Capacitors/CL10A106MA8NRNC
- added L10: ~, footprints:CKCS3015-3.3uH/M-K01, symbol component_library:Inductors/CKCS3015-3.3uH/M-K01
- added R85, R95: ~, footprints:RESC1005X35N, symbol component_library:Resistors/0402WGF1002TCE
- added R87: ~, footprints:RESC1005X35N, symbol component_library:Resistors/0402WGF1000TCE
- added R88: ~, footprints:RESC1005X35N, symbol component_library:Resistors/0402WGF1003TCE
- added R89: ~, footprints:RESC1005X35N, symbol component_library:Resistors/0402WGF2003TCE
- added R90: ~, footprints:RESC1005X35N, symbol component_library:Resistors/0402WGF1202TCE
- added R91: ~, footprints:RESC1608X45N, symbol component_library:Resistors/0603WAF1802T5E
- added R92: ~, footprints:RESC1005X35N, symbol component_library:Resistors/0402WGF1183TCE
- added R93: ~, footprints:RESC1608X45N, symbol component_library:Resistors/0603WAF3002T5E
- added R94: ~, footprints:RESC1608X45N, symbol component_library:Resistors/0603WAF3901T5E
- added U10: SY8088AAC, footprints:, symbol component_library:PMIC/SY8088AAC
- added U11: TPS7A0309PDBVR, footprints:, symbol component_library:PMIC/TPS7A0309PDBVR
- added U9: TLV75530PDBVR, footprints:, symbol component_library:PMIC/TLV75530PDBVR
Connections:
- net +1V8_VCC: now also R94.1, R95.1
- net +3V0_VCC: now also R93.1
- net +3V3_VCC_SYS: now also C192.1, C196.1, C197.1, C232.1, R85.1, U11.1 (IN), U9.1 (IN)
- net +5V0_SYS: now also C241.1, C242.1, U10.4 (IN)
- net GND: now also C192.2, C193.2, C194.2, C195.2, C196.2, C197.2, C232.2, C233.2, C234.2, C235.2, C236.2, C237.2, C238.2, C240.2, C241.2, C242.2, C243.2, R89.2, R90.2, U10.2 (GND), U11.2 (GND), U11.6 (GND_PAD), U9.2 (GND), U9.6 (GND_PAD)
- new net: C243.1, R95.2, U10.1 (EN)
- new net: C240.1, R90.1, R91.2, R92.1
- new net: R85.2, U11.3 (EN)
- new net +0V9_AVCC: C233.1, C234.1, C235.1, U11.5 (OUT)
- new net +0V9_VDD_LOG: C236.1, C237.1, C238.1, C239.1, L10.2, R87.1, R87.2, R88.1
- new net +3V0_VCC_SD: C193.1, C194.1, C195.1, U9.5 (OUT)
- new net 0V9_VDD_LOG_DVS_PWR_PWM: R91.1, R93.2, R94.2
- new net 0V9_VDD_LOG_FB: C239.2, R88.2, R89.1, R92.2, U10.5 (FB)
- new net 0V9_VDD_LOG_SW: L10.1, U10.3 (LX)
- new net 3V3_VCC_SD_EN: U9.3 (EN)
Other:
- note added: "Power of +0V9_AVCC"
- note added: "Power of +0V9_VDD_LOG"
- note added: "Power of +3V0_VCC_SD"
- note added: "Trace > 100mA"
- note added: "Trace > 500mA"
- moved on the sheet: C164, C165, C166, C167, C168, C169, C170, C171, C172, C173, C174, C175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

Commit message: design USB-A
Other:
- note added: "Trace > 750mA"
Changed lines of the file:
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@@
+		)
+	)
+	(text "Trace > 750mA"
+		(exclude_from_sim no)
+		(at 384.81 527.05 0)
+		(effects
+			(font
+				(size 1.27 1.27)
+				(thickness 0.254)
+				(bold yes)
+				(italic yes)
+			)
+			(justify left)
 		)
 	)
@@
 		)
 	)
+	(text "Trace > 1A"
+		(exclude_from_sim no)
+		(at 542.29 527.05 0)
+		(effects
+			(font
+				(size 1.27 1.27)
+				(thickness 0.254)
+				(bold yes)
+				(italic yes)
+			)
+			(justify right)
+		)
+	)

Commit message: design DDR
Parts:
- added C291: ~, footprints:CAPC3216X160N, symbol component_library:Capacitors/FV31X223K102EEG
- added R150: ~, footprints:RESC3115X55N, symbol component_library:Resistors/1206W4F1004T5E
- BAT1: footprint footprints: -> footprints:CR1220-2
- C48: renamed from C198; footprint footprints: -> footprints:CAPC2012X115N
- C53: renamed from C203; footprint footprints: -> footprints:CAPC2012X115N
- C54: renamed from C204; footprint footprints: -> footprints:CAPC2012X115N
- C64: renamed from C206; footprint footprints: -> footprints:CAPC1608X80N
- C67: renamed from C208; footprint footprints: -> footprints:CAPC2012X115N
- C68: renamed from C209; footprint footprints: -> footprints:CAPC2012X115N
- C69: renamed from C210; footprint footprints: -> footprints:CAPC2012X115N
- C77: renamed from C218; footprint footprints: -> footprints:CAPC2012X115N
- C78: renamed from C219; footprint footprints: -> footprints:CAPC2012X115N
- C90: renamed from C223; footprint footprints: -> footprints:CAPC2012X115N
- C97: renamed from C229; footprint footprints: -> footprints:CAPC2012X115N
- CON4: renamed from CON2; footprint footprints: -> footprints:DC-091
- L2: renamed from L7; footprint footprints: -> footprints:IHLP2525EZER1R0M01
- R46: renamed from R114; footprint footprints: -> footprints:RESC2012X55N
- renumbered C182 to C100, C191 to C101, C189 to C102, C190 to C103, C186 to C104, C187 to C105, C183 to C106, C184 to C107, C185 to C108, C188 to C109, C1 to C110, C2 to C111, C3 to C112, C4 to C113, C5 to C114, C6 to C115, C7 to C116, C8 to C117, C9 to C118, C192 to C119, C196 to C120, C194 to C121, C195 to C122, C193 to C123, C10 to C124, C11 to C125, C12 to C126, C13 to C127, C14 to C128, C15 to C129, C16 to C130, C17 to C131, C18 to C132, C19 to C133, C20 to C134, C21 to C135, C22 to C136, C23 to C137, C24 to C138, C25 to C139, C26 to C140, C27 to C141, C28 to C142, C29 to C143, C30 to C144, C31 to C145, C32 to C146, C33 to C147, C197 to C148, C232 to C149, C233 to C150, C234 to C151, C235 to C152, C34 to C153, C35 to C154, C36 to C155, C37 to C156, C38 to C157, C39 to C158, C46 to C159, C40 to C160, C41 to C161, C42 to C162, C241 to C163, C242 to C164, C236 to C165, C237 to C166, C238 to C167, C43 to C168, C243 to C169, C239 to C170, C44 to C171, C45 to C172, C240 to C173, C199 to C49, C200 to C50, C201 to C51, C202 to C52, C164 to C55, C165 to C56, C166 to C57, C167 to C58, C168 to C59, C169 to C60, C170 to C61, C171 to C62, C205 to C63, C172 to C65, C207 to C66, C211 to C70, C212 to C71, C213 to C72, C214 to C73, C215 to C74, C216 to C75, C217 to C76, C220 to C79, C221 to C80, C173 to C81, C174 to C82, C175 to C83, C176 to C84, C177 to C85, C178 to C86, C179 to C87, C180 to C88, C222 to C89, C224 to C91, C225 to C92, C181 to C93, C226 to C94, C227 to C95, C228 to C96, C230 to C98, C231 to C99, D10 to D19, D11 to D20, D1 to D21, D2 to D22, D5 to D23, D3 to D24, D4 to D25, D6 to D26, L5 to L1, L6 to L3, L8 to L4, L9 to L5, L1 to L6, L2 to L7, L3 to L8, L4 to L9, R102 to R32, R103 to R33, R104 to R34, R105 to R35, R106 to R36, R107 to R37, R108 to R38, R79 to R39, R80 to R40, R109 to R41, R110 to R42, R111 to R43, R112 to R44, R113 to R45, R115 to R47, R116 to R48, R117 to R49, R118 to R50, R119 to R51, R81 to R52, R82 to R53, R120 to R54, R121 to R55, R122 to R56, R123 to R57, R124 to R58, R83 to R59, R84 to R60, R86 to R61, R1 to R62, R2 to R63, R3 to R64, R4 to R65, R5 to R66, R85 to R67, R6 to R68, R12 to R69, R13 to R70, R14 to R71, R7 to R72, R8 to R73, R9 to R74, R10 to R75, R87 to R76, R11 to R77, R95 to R78, R88 to R79, R91 to R80, R92 to R81, R90 to R82, R89 to R83, R94 to R84, R93 to R85, U4 to U10, U8 to U11, U5 to U12, U1 to U13, U9 to U14, U11 to U15, U10 to U16, U6 to U7, U3 to U8, U7 to U9
Connections:
- net GND: now also C291.2, R150.2
- new net CHGND: C291.1, CON4.SHIELD, R150.1
Other:
- moved on the sheet: C48, C49, C50, C51, C52, C53, C54, C63, C64, D19, D20, R32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
