File: RAM1.kicad_sch (KiCad schematic)
At the start: 0 parts

Commit message: design CPU-RK3399 eMMC Controller
Other:
- company: (none) -> TickLab
Changed lines of the file:
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@@
 	(paper "A4")
 	(title_block
-		(date "2026-01-09")
+		(date "2026-01-14")
 		(rev "1.0.0")
+		(company "TickLab")
 	)
 	(bus

Commit message: design DDR
Parts:
- added U20, U21: MT41K256M16TW-107:P, footprints:BGA96C80P9X16_800X1400X110, symbol component_library:ICs/MT41K256M16TW-107P
Connections:
- net CAS#: now also U20.K3 (~{CAS}), U21.K3 (~{CAS})
- net RAS#: now also U20.J3 (~{RAS}), U21.J3 (~{RAS})
- net RESET#: now also U20.T2 (~{RESET}), U21.T2 (~{RESET})
- net WE#: now also U20.L3 (~{WE}), U21.L3 (~{WE})
- new net +1V35_VCC_DDR: U20.A1 (VDDQ), U20.A8 (VDDQ), U20.B2 (VDD), U20.C1 (VDDQ), U20.C9 (VDDQ), U20.D2 (VDDQ), U20.D9 (VDD), U20.E9 (VDDQ), U20.F1 (VDDQ), U20.G7 (VDD), U20.H2 (VDDQ), U20.H9 (VDDQ), U20.K2 (VDD), U20.K8 (VDD), U20.N1 (VDD), U20.N9 (VDD), U20.R1 (VDD), U20.R9 (VDD), U21.A1 (VDDQ), U21.A8 (VDDQ), U21.B2 (VDD), U21.C1 (VDDQ), U21.C9 (VDDQ), U21.D2 (VDDQ), U21.D9 (VDD), U21.E9 (VDDQ), U21.F1 (VDDQ), U21.G7 (VDD), U21.H2 (VDDQ), U21.H9 (VDDQ), U21.K2 (VDD), U21.K8 (VDD), U21.N1 (VDD), U21.N9 (VDD), U21.R1 (VDD), U21.R9 (VDD)
- new net GND: U20.A9 (VSS), U20.B1 (VSSQ), U20.B3 (VSS), U20.B9 (VSSQ), U20.D1 (VSSQ), U20.D8 (VSSQ), U20.E1 (VSS), U20.E2 (VSSQ), U20.E8 (VSSQ), U20.F9 (VSSQ), U20.G1 (VSSQ), U20.G8 (VSS), U20.G9 (VSSQ), U20.J2 (VSS), U20.J8 (VSS), U20.M1 (VSS), U20.M9 (VSS), U20.P1 (VSS), U20.P9 (VSS), U20.T1 (VSS), U20.T9 (VSS), U21.A9 (VSS), U21.B1 (VSSQ), U21.B3 (VSS), U21.B9 (VSSQ), U21.D1 (VSSQ), U21.D8 (VSSQ), U21.E1 (VSS), U21.E2 (VSSQ), U21.E8 (VSSQ), U21.F9 (VSSQ), U21.G1 (VSSQ), U21.G8 (VSS), U21.G9 (VSSQ), U21.J2 (VSS), U21.J8 (VSS), U21.M1 (VSS), U21.M9 (VSS), U21.P1 (VSS), U21.P9 (VSS), U21.T1 (VSS), U21.T9 (VSS)
- new net RAM1_A0: U20.N3 (A0), U21.N3 (A0)
- new net RAM1_A1: U20.P7 (A1), U21.P7 (A1)
- new net RAM1_A10: U20.L7 (A10/AP), U21.L7 (A10/AP)
- new net RAM1_A11: U20.R7 (A11), U21.R7 (A11)
- new net RAM1_A12: U20.N7 (A12/~{BC}), U21.N7 (A12/~{BC})
- new net RAM1_A13: U20.T3 (A13), U21.T3 (A13)
- new net RAM1_A14: U20.T7 (A14), U21.T7 (A14)
- new net RAM1_A15: U20.M7 (NC), U21.M7 (NC)
- new net RAM1_A2: U20.P3 (A2), U21.P3 (A2)
- new net RAM1_A3: U20.N2 (A3), U21.N2 (A3)
- new net RAM1_A4: U20.P8 (A4), U21.P8 (A4)
- new net RAM1_A5: U20.P2 (A5), U21.P2 (A5)
- new net RAM1_A6: U20.R8 (A6), U21.R8 (A6)
- new net RAM1_A7: U20.R2 (A7), U21.R2 (A7)
- new net RAM1_A8: U20.T8 (A8), U21.T8 (A8)
- new net RAM1_A9: U20.R3 (A9), U21.R3 (A9)
- new net RAM1_BA0: U20.M2 (BA0), U21.M2 (BA0)
- new net RAM1_BA1: U20.N8 (BA1), U21.N8 (BA1)
- new net RAM1_BA2: U20.M3 (BA2), U21.M3 (BA2)
- new net RAM1_CKE0: U20.K9 (CKE), U21.K9 (CKE)
- new net RAM1_CKE1: U20.J9 (NC), U21.J9 (NC)
- new net RAM1_CLK0+: U20.J7 (CK), U21.J7 (CK)
- new net RAM1_CLK0-: U20.K7 (~{CK}), U21.K7 (~{CK})
- new net RAM1_CS#0: U20.L2 (~{CS}), U21.L2 (~{CS})
- new net RAM1_CS#1: U20.L1 (NC), U21.L1 (NC)
- new net RAM1_DM0: U20.E7 (LDM)
- new net RAM1_DM1: U21.E7 (LDM)
- new net RAM1_DM2: U20.D3 (UDM)
- new net RAM1_DM3: U21.D3 (UDM)
- new net RAM1_DQ0: U20.E3 (DQ0)
- new net RAM1_DQ1: U20.F7 (DQ1)
- new net RAM1_DQ10: U20.C8 (DQ10)
- new net RAM1_DQ11: U20.C2 (DQ11)
- new net RAM1_DQ12: U20.A7 (DQ12)
- new net RAM1_DQ13: U20.A2 (DQ13)
- new net RAM1_DQ14: U20.B8 (DQ14)
- new net RAM1_DQ15: U20.A3 (DQ15)
- new net RAM1_DQ16: U21.E3 (DQ0)
- new net RAM1_DQ17: U21.F7 (DQ1)
- new net RAM1_DQ18: U21.F2 (DQ2)
- new net RAM1_DQ19: U21.F8 (DQ3)
- new net RAM1_DQ2: U20.F2 (DQ2)
- new net RAM1_DQ20: U21.H3 (DQ4)
- new net RAM1_DQ21: U21.H8 (DQ5)
- new net RAM1_DQ22: U21.G2 (DQ6)
- new net RAM1_DQ23: U21.H7 (DQ7)
- new net RAM1_DQ24: U21.D7 (DQ8)
- new net RAM1_DQ25: U21.C3 (DQ9)
- new net RAM1_DQ26: U21.C8 (DQ10)
- new net RAM1_DQ27: U21.C2 (DQ11)
- new net RAM1_DQ28: U21.A7 (DQ12)
- new net RAM1_DQ29: U21.A2 (DQ13)
- new net RAM1_DQ3: U20.F8 (DQ3)
- new net RAM1_DQ30: U21.B8 (DQ14)
- new net RAM1_DQ31: U21.A3 (DQ15)
- new net RAM1_DQ4: U20.H3 (DQ4)
- new net RAM1_DQ5: U20.H8 (DQ5)
- new net RAM1_DQ6: U20.G2 (DQ6)
- new net RAM1_DQ7: U20.H7 (DQ7)
- new net RAM1_DQ8: U20.D7 (DQ8)
- new net RAM1_DQ9: U20.C3 (DQ9)
- new net RAM1_DQS0+: U20.F3 (LDQS)
- new net RAM1_DQS0-: U20.G3 (~{LDQS})
- new net RAM1_DQS1+: U21.F3 (LDQS)
- new net RAM1_DQS1-: U21.G3 (~{LDQS})
- new net RAM1_DQS2+: U20.C7 (UDQS)
- new net RAM1_DQS2-: U20.B7 (~{UDQS})
- new net RAM1_DQS3+: U21.C7 (UDQS)
- new net RAM1_DQS3-: U21.B7 (~{UDQS})
- new net RAM1_ODT0: U20.K1 (ODT), U21.K1 (ODT)
- new net RAM1_ODT1: U20.J1 (NC), U21.J1 (NC)
