File: Recovery_Button.kicad_sch (KiCad schematic)
At the start: 5 parts

Commit message: design PMIC
Changed lines of the file:
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@@
 		(rev "1.0.0")
 		(company "TickLab")
-		(comment 1 "Project: VESA-SBC3399")
+		(comment 1 "VESA-SBC3399")
 	)
 	(junction

Commit message: update design power
Parts:
- renumbered BTN1 to BTN3, C103 to C158, D1 to D7, R27 to R50, R28 to R51
Changed lines of the file:
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@@
 		(dnp no)
 		(fields_autoplaced yes)
-		(property "Reference" "#PWR0107"
+		(property "Reference" "#PWR0194"
 			(at 154.94 120.65 0)
 			(effects
@@
 			(project "VESA-SBC3399"
 				(path "/ebc9dc57-8b05-484a-a5cd-c53b1efc71d3/330777a9-95d0-480d-9a4e-ca1348364667"
-					(reference "#PWR0107")
+					(reference "#PWR0194")
 					(unit 1)
 				)
@@
 		(on_board yes)
 		(dnp no)
-		(property "Reference" "C103"
+		(property "Reference" "C158"
 			(at 146.05 104.1399 0)
 			(effects
@@
 			(project ""
 				(path "/ebc9dc57-8b05-484a-a5cd-c53b1efc71d3/330777a9-95d0-480d-9a4e-ca1348364667"
-					(reference "C103")
+					(reference "C158")
 					(unit 1)
 				)
@@
 		(dnp no)
 		(fields_autoplaced yes)
-		(property "Reference" "R28"
+		(property "Reference" "R51"
 			(at 135.89 92.71 0)
 			(effects
@@
 			(project ""
 				(path "/ebc9dc57-8b05-484a-a5cd-c53b1efc71d3/330777a9-95d0-480d-9a4e-ca1348364667"
-					(reference "R28")
+					(reference "R51")
 					(unit 1)
 				)
@@
 		(dnp no)
 		(fields_autoplaced yes)
-		(property "Reference" "R27"
+		(property "Reference" "R50"
 			(at 144.78 92.7099 90)
 			(effects
@@
 			(project ""
 				(path "/ebc9dc57-8b05-484a-a5cd-c53b1efc71d3/330777a9-95d0-480d-9a4e-ca1348364667"
-					(reference "R27")
+					(reference "R50")
 					(unit 1)
 				)
@@
 		(on_board yes)
 		(dnp no)
-		(property "Reference" "#PWR0104"
+		(property "Reference" "#PWR0191"
 			(at 142.24 92.71 0)
 			(effects
@@
 			(project "VESA-SBC3399"
 				(path "/ebc9dc57-8b05-484a-a5cd-c53b1efc71d3/330777a9-95d0-480d-9a4e-ca1348364667"
-					(reference "#PWR0104")
+					(reference "#PWR0191")
 					(unit 1)
 				)
@@
 		(dnp no)
 		(fields_autoplaced yes)
-		(property "Reference" "#PWR0106"
+		(property "Reference" "#PWR0193"
 			(at 142.24 120.65 0)
 			(effects
@@
 			(project "VESA-SBC3399"
 				(path "/ebc9dc57-8b05-484a-a5cd-c53b1efc71d3/330777a9-95d0-480d-9a4e-ca1348364667"
-					(reference "#PWR0106")
+					(reference "#PWR0193")
 					(unit 1)
 				)
@@
 		(dnp no)
 		(fields_autoplaced yes)
-		(property "Reference" "D1"
+		(property "Reference" "D7"
 			(at 157.48 106.4259 0)
 			(effects
@@
 			(project ""
 				(path "/ebc9dc57-8b05-484a-a5cd-c53b1efc71d3/330777a9-95d0-480d-9a4e-ca1348364667"
-					(reference "D1")
+					(reference "D7")
 					(unit 1)
 				)
@@
 		(dnp no)
 		(fields_autoplaced yes)
-		(property "Reference" "BTN1"
+		(property "Reference" "BTN3"
 			(at 121.92 93.98 0)
 			(effects
@@
 			(project ""
 				(path "/ebc9dc57-8b05-484a-a5cd-c53b1efc71d3/330777a9-95d0-480d-9a4e-ca1348364667"
-					(reference "BTN1")
+					(reference "BTN3")
 					(unit 1)
 				)
@@
 		(dnp no)
 		(fields_autoplaced yes)
-		(property "Reference" "#PWR0105"
+		(property "Reference" "#PWR0192"
 			(at 114.3 113.03 0)
 			(effects
@@
 			(project "VESA-SBC3399"
 				(path "/ebc9dc57-8b05-484a-a5cd-c53b1efc71d3/330777a9-95d0-480d-9a4e-ca1348364667"
-					(reference "#PWR0105")
+					(reference "#PWR0192")
 					(unit 1)
 				)

Commit message: design DDR
Parts:
- renumbered C158 to C285, D7 to D27, R50 to R121, R51 to R122
Changed lines of the file:
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@@
 		(dnp no)
 		(fields_autoplaced yes)
-		(property "Reference" "#PWR0194"
+		(property "Reference" "#PWR0354"
 			(at 154.94 120.65 0)
 			(effects
@@
 			(project "VESA-SBC3399"
 				(path "/ebc9dc57-8b05-484a-a5cd-c53b1efc71d3/330777a9-95d0-480d-9a4e-ca1348364667"
-					(reference "#PWR0194")
+					(reference "#PWR0354")
 					(unit 1)
 				)
@@
 		(on_board yes)
 		(dnp no)
-		(property "Reference" "C158"
+		(property "Reference" "C285"
 			(at 146.05 104.1399 0)
 			(effects
@@
 			(project ""
 				(path "/ebc9dc57-8b05-484a-a5cd-c53b1efc71d3/330777a9-95d0-480d-9a4e-ca1348364667"
-					(reference "C158")
+					(reference "C285")
 					(unit 1)
 				)
@@
 		(dnp no)
 		(fields_autoplaced yes)
-		(property "Reference" "R51"
+		(property "Reference" "R122"
 			(at 135.89 92.71 0)
 			(effects
@@
 			(project ""
 				(path "/ebc9dc57-8b05-484a-a5cd-c53b1efc71d3/330777a9-95d0-480d-9a4e-ca1348364667"
-					(reference "R51")
+					(reference "R122")
 					(unit 1)
 				)
@@
 		(dnp no)
 		(fields_autoplaced yes)
-		(property "Reference" "R50"
+		(property "Reference" "R121"
 			(at 144.78 92.7099 90)
 			(effects
@@
 			(project ""
 				(path "/ebc9dc57-8b05-484a-a5cd-c53b1efc71d3/330777a9-95d0-480d-9a4e-ca1348364667"
-					(reference "R50")
+					(reference "R121")
 					(unit 1)
 				)
@@
 		(on_board yes)
 		(dnp no)
-		(property "Reference" "#PWR0191"
+		(property "Reference" "#PWR0351"
 			(at 142.24 92.71 0)
 			(effects
@@
 			(project "VESA-SBC3399"
 				(path "/ebc9dc57-8b05-484a-a5cd-c53b1efc71d3/330777a9-95d0-480d-9a4e-ca1348364667"
-					(reference "#PWR0191")
+					(reference "#PWR0351")
 					(unit 1)
 				)
@@
 		(dnp no)
 		(fields_autoplaced yes)
-		(property "Reference" "#PWR0193"
+		(property "Reference" "#PWR0353"
 			(at 142.24 120.65 0)
 			(effects
@@
 			(project "VESA-SBC3399"
 				(path "/ebc9dc57-8b05-484a-a5cd-c53b1efc71d3/330777a9-95d0-480d-9a4e-ca1348364667"
-					(reference "#PWR0193")
+					(reference "#PWR0353")
 					(unit 1)
 				)
@@
 		(dnp no)
 		(fields_autoplaced yes)
-		(property "Reference" "D7"
+		(property "Reference" "D27"
 			(at 157.48 106.4259 0)
 			(effects
@@
 			(project ""
 				(path "/ebc9dc57-8b05-484a-a5cd-c53b1efc71d3/330777a9-95d0-480d-9a4e-ca1348364667"
-					(reference "D7")
+					(reference "D27")
 					(unit 1)
 				)
@@
 		(dnp no)
 		(fields_autoplaced yes)
-		(property "Reference" "#PWR0192"
+		(property "Reference" "#PWR0352"
 			(at 114.3 113.03 0)
 			(effects
@@
 			(project "VESA-SBC3399"
 				(path "/ebc9dc57-8b05-484a-a5cd-c53b1efc71d3/330777a9-95d0-480d-9a4e-ca1348364667"
-					(reference "#PWR0192")
+					(reference "#PWR0352")
 					(unit 1)
 				)
