File: USBA.kicad_sch (KiCad schematic)
At the start: 15 parts, among them CON1 AF SS-JB17.6

Commit message: design DDR
Parts:
- removed R100, R97, R98, R99: ~, footprints:RESC1005X35N, symbol component_library:Resistors/0402WGF220JTCE
- added C42, C45: ~, footprints:CAPC1005X50N, symbol component_library:Capacitors/CL05B104KO5NNNC
- added C43, C46: ~, footprints:CAPC1005X50N, symbol component_library:Capacitors/0402CG180J500NT
- added C44, C47: ~, footprints:CAPC1608X80N, symbol component_library:Capacitors/CL10A106MA8NRNC
- added R23, R24, R25, R26: ~, footprints:RESC1005X35N, symbol component_library:Resistors/CQ02WGF220KTCE
- added R28, R30: ~, footprints:RESC1005X35N, symbol component_library:Resistors/0402WGF1003TCE
- added R29, R31: ~, footprints:RESC1608X45N, symbol component_library:Resistors/0603WAF9101T5E
- added U5, U6: SY6280AAC, footprints:, symbol component_library:PMIC/SY6280AAC
- renumbered C245 to C37, C247 to C38, C246 to C39, C248 to C40, C244 to C41, CON1 to CON3, D12 to D15, D13 to D16, D8 to D17, D9 to D18, R96 to R27
Connections:
- net +5V0_VBUS_USBA0: now also C43.1, C44.1, U5.1 (OUT)
- net +5V0_VBUS_USBA1: now also C46.1, C47.1, U6.1 (OUT)
- net CHGND: now also C41.1, R27.1; no longer C41.2, R27.2
- net GND: now also C41.2, R27.2, C42.2, C43.2, C44.2, C45.2, C46.2, C47.2, R28.2, R29.2, R30.2, R31.2, U5.2 (GND), U6.2 (GND); no longer C41.1, R27.1
- net USBA0_D+: now also R23.1
- net USBA0_D-: now also R24.1
- net USBA0_D_R+: now also R23.2
- net USBA0_D_R-: now also R24.2
- net USBA1_D+: now also R25.1
- net USBA1_D-: now also R26.1
- net USBA1_D_R+: now also R25.2
- net USBA1_D_R-: now also R26.2
- new net: R31.1, U6.3 (ISET)
- new net: R29.1, U5.3 (ISET)
- new net +5V0_USB: C42.1, C45.1, U5.5 (IN), U6.5 (IN)
- new net VBUS_USBA_EN: R28.1, R30.1, U5.4 (EN), U6.4 (EN)
Other:
- note added: "Trace > 750mA"
- note added: "USB 2.0 Type-A Host Port"
- note added: "USB Type-A Power Switch"
- moved on the sheet: C37, C38, C39, C40, C41, CON3, D15, D16, R27
