File: USBC0.kicad_sch (KiCad schematic)
At the start: 0 parts

Commit message: design CPU-RK3399 eMMC Controller
Other:
- company: (none) -> TickLab
Changed lines of the file:
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@@
 	(paper "A4")
 	(title_block
-		(date "2026-01-09")
+		(date "2026-01-14")
 		(rev "1.0.0")
+		(company "TickLab")
 	)
 	(bus

Commit message: design DDR
Parts:
- added C1, C11, C12, C14, C2, C3, C4, C5, C7, C8, C9: ~, footprints:CAPC1005X50N, symbol component_library:Capacitors/CL05B104KO5NNNC
- added C10: ~, footprints:CAPC1005X50N, symbol component_library:Capacitors/CL05A105KA5NQNC
- added C13: ~, footprints:CAPC1005X50N, symbol component_library:Capacitors/0402CG180J500NT
- added C15: ~, footprints:CAPC2012X115N, symbol component_library:Capacitors/CL21A226MAQNNNE
- added C16: ~, footprints:CAPC1005X50N, symbol component_library:Capacitors/0402CG330J500NT
- added C17, C18: ~, footprints:CAPC1005X50N, symbol component_library:Capacitors/0402B221K500NT
- added C6: ~, footprints:CAPC3216X160N, symbol component_library:Capacitors/FV31X223K102EEG
- added CON1: ~, footprints:TYPE-C 24P QT, symbol component_library:Connectors/TYPE-C 24P QT
- added D1, D2, D3: ~, footprints:, symbol component_library:TVS, ESD/ESD5302F
- added D4, D5: ~, footprints:, symbol component_library:TVS, ESD/TPD4E05U06DQAR
- added D6, D7: ~, footprints:, symbol component_library:TVS, ESD/SMF5.0A
- added R1, R2: ~, footprints:RESC1608X45N, symbol component_library:Resistors/0603WAF2004T5E
- added R10, R11, R3, R4: ~, footprints:RESC1005X35N, symbol component_library:Resistors/0402WGF1003TCE
- added R5: ~, footprints:RESC1005X35N, symbol component_library:Resistors/0402WGF1002TCE
- added R6, R8: ~, footprints:RESC1005X35N, symbol component_library:Resistors/CQ02WGF220KTCE
- added R7: ~, footprints:RESC1005X35N, symbol component_library:Resistors/0402WGF1502TCE
- added R9: ~, footprints:RESC3115X55N, symbol component_library:Resistors/1206W4F1004T5E
- added U1: TPS259261DRCR, symbol component_library_symbols:TPS259261DRCR
- added U2: FUSB302BMPX, symbol component_library_symbols:FUSB302BMPX
Connections:
- net INT#: now also U2.5 (INT_N)
- new net: C16.1, U1.1 (dV/dT)
- new net: R11.1, U1.10 (ILIM)
- new net +3V3_VCC_SYS: C11.1, U2.3 (VDD), U2.4 (VDD)
- new net +5V0_USB: C10.1, C12.1, C9.1, D6.C (Cathode), U1.3 (VIN), U1.4 (VIN), U1.5 (VIN), U2.12 (VCONN), U2.13 (VCONN)
- new net +5V0_VBUS_USBC0: C13.1, C14.1, C15.1, CON1.A4 (VBUS), CON1.A9 (VBUS), CON1.B4 (VBUS), CON1.B9 (VBUS), D7.C (Cathode), R5.1, U1.6 (OUT), U1.7 (OUT), U1.8 (OUT), U2.2 (VBUS)
- new net CHGND: C6.1, CON1.1 (SHIELD), CON1.2 (SHIELD), CON1.3 (SHIELD), CON1.4 (SHIELD), R9.1
- new net CPU_I2C4_SCL: U2.6 (SCL)
- new net CPU_I2C4_SDA: U2.7 (SDA)
- new net GND: C10.2, C11.2, C12.2, C13.2, C14.2, C15.2, C16.2, C17.2, C18.2, C3.2, C6.2, C9.2, CON1.A1 (GND), CON1.A12 (GND), CON1.B1 (GND), CON1.B12 (GND), D1.3, D2.3, D3.3, D4.3 (GND), D4.8 (GND), D5.3 (GND), D5.8 (GND), D6.A (Anode), D7.A (Anode), R1.2, R10.2, R11.2, R2.2, R7.2, R9.2, U1.11 (PAD_GND), U2.15 (PAD_GND), U2.8 (GND), U2.9 (GND)
- new net USBC0_CC1: C17.1, CON1.A5 (CC1), D2.1, U2.10 (CC1), U2.11 (CC1)
- new net USBC0_CC2: C18.1, CON1.B5 (CC2), D2.2, U2.1 (CC2), U2.14 (CC2)
- new net USBC0_D+: R6.1
- new net USBC0_D-: R8.1
- new net USBC0_DC_SBUS1: R3.1
- new net USBC0_DC_SBUS2: R4.1
- new net USBC0_D_R+: CON1.A6 (D1+), CON1.B6 (D2+), D3.1, R6.2
- new net USBC0_D_R-: CON1.A7 (D1-), CON1.B7 (D2-), D3.2, R8.2
- new net USBC0_RX1+: CON1.B11 (RX1+), D4.4 (D2+), D4.7 (NC)
- new net USBC0_RX1-: CON1.B10 (RX1-), D4.5 (D2-), D4.6 (NC)
- new net USBC0_RX2+: CON1.A11 (RX2+), D5.4 (D2+), D5.7 (NC)
- new net USBC0_RX2-: CON1.A10 (RX2-), D5.5 (D2-), D5.6 (NC)
- new net USBC0_SBUS1: C1.1
- new net USBC0_SBUS1_C: C1.2, CON1.A8 (SBUS1), D1.1, R1.1, R3.2
- new net USBC0_SBUS2: C2.1
- new net USBC0_SBUS2_C: C2.2, CON1.B8 (SBUS2), D1.2, R2.1, R4.2
- new net USBC0_TX1+: C4.1
- new net USBC0_TX1-: C5.1
- new net USBC0_TX1_C+: C4.2, CON1.A2 (TX1+), D4.1 (D1+), D4.10 (NC)
- new net USBC0_TX1_C-: C5.2, CON1.A3 (TX1-), D4.2 (D1-), D4.9 (NC)
- new net USBC0_TX2+: C7.1
- new net USBC0_TX2-: C8.1
- new net USBC0_TX2_C+: C7.2, CON1.B2 (TX2+), D5.1 (D1+), D5.10 (NC)
- new net USBC0_TX2_C-: C8.2, CON1.B3 (TX2-), D5.2 (D1-), D5.9 (NC)
- new net VBUS_USBC0_VBUSDET: C3.1, R5.2, R7.1
- new net VBUS_USBC_EN: R10.1, U1.2 (EN/UVLO)
Other:
- note added: "Trace > 3A"
- note added: "USB 3.0 Type-C0 displayPort"
- note added: "USB Type-C0 CC Controller"
- note added: "USB Type-C0 Power Switch"
- title: (none) -> USB 3.0 Type-C0
