File: USBC1.kicad_sch (KiCad schematic)
At the start: 0 parts

Commit message: design CPU-RK3399 eMMC Controller
Other:
- company: (none) -> TickLab
Changed lines of the file:
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@@
 	(paper "A4")
 	(title_block
-		(date "2026-01-09")
+		(date "2026-01-14")
 		(rev "1.0.0")
+		(company "TickLab")
 	)
 	(bus

Commit message: design DDR
Parts:
- added C19, C20, C21, C22, C23, C25, C26, C27, C29, C30, C32: ~, footprints:CAPC1005X50N, symbol component_library:Capacitors/CL05B104KO5NNNC
- added C24: ~, footprints:CAPC3216X160N, symbol component_library:Capacitors/FV31X223K102EEG
- added C28: ~, footprints:CAPC1005X50N, symbol component_library:Capacitors/CL05A105KA5NQNC
- added C31: ~, footprints:CAPC1005X50N, symbol component_library:Capacitors/0402CG180J500NT
- added C33: ~, footprints:CAPC2012X115N, symbol component_library:Capacitors/CL21A226MAQNNNE
- added C34: ~, footprints:CAPC1005X50N, symbol component_library:Capacitors/0402CG330J500NT
- added C35, C36: ~, footprints:CAPC1005X50N, symbol component_library:Capacitors/0402B221K500NT
- added CON2: ~, footprints:TYPE-C 24P QT, symbol component_library:Connectors/TYPE-C 24P QT
- added D10, D8, D9: ~, footprints:, symbol component_library:TVS, ESD/ESD5302F
- added D11, D12: ~, footprints:, symbol component_library:TVS, ESD/TPD4E05U06DQAR
- added D13, D14: ~, footprints:, symbol component_library:TVS, ESD/SMF5.0A
- added R12, R13: ~, footprints:RESC1608X45N, symbol component_library:Resistors/0603WAF2004T5E
- added R14, R15, R21, R22: ~, footprints:RESC1005X35N, symbol component_library:Resistors/0402WGF1003TCE
- added R16: ~, footprints:RESC1005X35N, symbol component_library:Resistors/0402WGF1002TCE
- added R17, R19: ~, footprints:RESC1005X35N, symbol component_library:Resistors/CQ02WGF220KTCE
- added R18: ~, footprints:RESC1005X35N, symbol component_library:Resistors/0402WGF1502TCE
- added R20: ~, footprints:RESC3115X55N, symbol component_library:Resistors/1206W4F1004T5E
- added U3: TPS259261DRCR, symbol component_library_symbols:TPS259261DRCR
- added U4: FUSB302BMPX, symbol component_library_symbols:FUSB302BMPX
Connections:
- net INT#: now also U4.5 (INT_N)
- new net: R22.1, U3.10 (ILIM)
- new net: C34.1, U3.1 (dV/dT)
- new net +3V3_VCC_SYS: C29.1, U4.3 (VDD), U4.4 (VDD)
- new net +5V0_USB: C27.1, C28.1, C30.1, D13.C (Cathode), U3.3 (VIN), U3.4 (VIN), U3.5 (VIN), U4.12 (VCONN), U4.13 (VCONN)
- new net +5V0_VBUS_USBC1: C31.1, C32.1, C33.1, CON2.A4 (VBUS), CON2.A9 (VBUS), CON2.B4 (VBUS), CON2.B9 (VBUS), D14.C (Cathode), R16.1, U3.6 (OUT), U3.7 (OUT), U3.8 (OUT), U4.2 (VBUS)
- new net CHGND: C24.1, CON2.1 (SHIELD), CON2.2 (SHIELD), CON2.3 (SHIELD), CON2.4 (SHIELD), R20.1
- new net CPU_I2C4_SCL: U4.6 (SCL)
- new net CPU_I2C4_SDA: U4.7 (SDA)
- new net GND: C21.2, C24.2, C27.2, C28.2, C29.2, C30.2, C31.2, C32.2, C33.2, C34.2, C35.2, C36.2, CON2.A1 (GND), CON2.A12 (GND), CON2.B1 (GND), CON2.B12 (GND), D10.3, D11.3 (GND), D11.8 (GND), D12.3 (GND), D12.8 (GND), D13.A (Anode), D14.A (Anode), D8.3, D9.3, R12.2, R13.2, R18.2, R20.2, R21.2, R22.2, U3.11 (PAD_GND), U4.15 (PAD_GND), U4.8 (GND), U4.9 (GND)
- new net USBC1_CC1: C35.1, CON2.A5 (CC1), D9.1, U4.10 (CC1), U4.11 (CC1)
- new net USBC1_CC2: C36.1, CON2.B5 (CC2), D9.2, U4.1 (CC2), U4.14 (CC2)
- new net USBC1_D+: R17.1
- new net USBC1_D-: R19.1
- new net USBC1_DC_SBUS1: R14.1
- new net USBC1_DC_SBUS2: R15.1
- new net USBC1_D_R+: CON2.A6 (D1+), CON2.B6 (D2+), D10.1, R17.2
- new net USBC1_D_R-: CON2.A7 (D1-), CON2.B7 (D2-), D10.2, R19.2
- new net USBC1_RX1+: CON2.B11 (RX1+), D11.4 (D2+), D11.7 (NC)
- new net USBC1_RX1-: CON2.B10 (RX1-), D11.5 (D2-), D11.6 (NC)
- new net USBC1_RX2+: CON2.A11 (RX2+), D12.4 (D2+), D12.7 (NC)
- new net USBC1_RX2-: CON2.A10 (RX2-), D12.5 (D2-), D12.6 (NC)
- new net USBC1_SBUS1: C19.1
- new net USBC1_SBUS1_C: C19.2, CON2.A8 (SBUS1), D8.1, R12.1, R14.2
- new net USBC1_SBUS2: C20.1
- new net USBC1_SBUS2_C: C20.2, CON2.B8 (SBUS2), D8.2, R13.1, R15.2
- new net USBC1_TX1+: C22.1
- new net USBC1_TX1-: C23.1
- new net USBC1_TX1_C+: C22.2, CON2.A2 (TX1+), D11.1 (D1+), D11.10 (NC)
- new net USBC1_TX1_C-: C23.2, CON2.A3 (TX1-), D11.2 (D1-), D11.9 (NC)
- new net USBC1_TX2+: C25.1
- new net USBC1_TX2-: C26.1
- new net USBC1_TX2_C+: C25.2, CON2.B2 (TX2+), D12.1 (D1+), D12.10 (NC)
- new net USBC1_TX2_C-: C26.2, CON2.B3 (TX2-), D12.2 (D1-), D12.9 (NC)
- new net VBUS_USBC1_VBUSDET: C21.1, R16.2, R18.1
- new net VBUS_USBC_EN: R21.1, U3.2 (EN/UVLO)
Other:
- note added: "Trace > 3A"
- note added: "USB 3.0 Type-C1 displayPort"
- note added: "USB Type-C1 CC Controller"
- note added: "USB Type-C1 Power Switch"
