File: _autosave-VESA-SBC3399.kicad_pcb (KiCad board)
At the start: 2 copper layers, 85 x 85 mm, 410 parts, among them CON3 AF SS-JB17.6, U17 RK3399, U18 MT41K256M16TW-107:P, U19 MT41K256M16TW-107:P, U20 MT41K256M16TW-107:P, U21 MT41K256M16TW-107:P

Commit message: design DDR
Parts:
- moved U20 34.8 mm to (72.6, 119.2)
- moved U21 27.3 mm to (63.6, 119.2), turned to 0 degrees
- moved U18 25.3 mm to (64.6, 102.2), turned to 0 degrees
- moved U19 10.2 mm to (73.2, 102.2), turned to 0 degrees
Connections:
- U18 pad L7: unconnected-(U18-A10/AP-PadL7) -> /RAM0_A10
- U18 pad N2: unconnected-(U18-A3-PadN2) -> /RAM0_A3
- U18 pad N3: unconnected-(U18-A0-PadN3) -> /RAM0_A0
- U18 pad N7: unconnected-(U18-A12/~{BC}-PadN7) -> /RAM0_A12
- U18 pad P2: unconnected-(U18-A5-PadP2) -> /RAM0_A5
- U18 pad P3: unconnected-(U18-A2-PadP3) -> /RAM0_A2
- U18 pad P7: unconnected-(U18-A1-PadP7) -> /RAM0_A1
- U18 pad P8: unconnected-(U18-A4-PadP8) -> /RAM0_A4
- U18 pad R2: unconnected-(U18-A7-PadR2) -> /RAM0_A7
- U18 pad R3: unconnected-(U18-A9-PadR3) -> /RAM0_A9
- U18 pad R7: unconnected-(U18-A11-PadR7) -> /RAM0_A11
- U18 pad R8: unconnected-(U18-A6-PadR8) -> /RAM0_A6
- U18 pad T3: unconnected-(U18-A13-PadT3) -> /RAM0_A13
- U18 pad T7: unconnected-(U18-A14-PadT7) -> /RAM0_A14
- U18 pad T8: unconnected-(U18-A8-PadT8) -> /RAM0_A8
- U19 pad L7: unconnected-(U19-A10/AP-PadL7) -> /RAM0_A10
- U19 pad N2: unconnected-(U19-A3-PadN2) -> /RAM0_A3
- U19 pad N3: unconnected-(U19-A0-PadN3) -> /RAM0_A0
- U19 pad N7: unconnected-(U19-A12/~{BC}-PadN7) -> /RAM0_A12
- U19 pad P2: unconnected-(U19-A5-PadP2) -> /RAM0_A5
- U19 pad P3: unconnected-(U19-A2-PadP3) -> /RAM0_A2
- U19 pad P7: unconnected-(U19-A1-PadP7) -> /RAM0_A1
- U19 pad P8: unconnected-(U19-A4-PadP8) -> /RAM0_A4
- U19 pad R2: unconnected-(U19-A7-PadR2) -> /RAM0_A7
- U19 pad R3: unconnected-(U19-A9-PadR3) -> /RAM0_A9
- U19 pad R7: unconnected-(U19-A11-PadR7) -> /RAM0_A11
- U19 pad R8: unconnected-(U19-A6-PadR8) -> /RAM0_A6
- U19 pad T3: unconnected-(U19-A13-PadT3) -> /RAM0_A13
- U19 pad T7: unconnected-(U19-A14-PadT7) -> /RAM0_A14
- U19 pad T8: unconnected-(U19-A8-PadT8) -> /RAM0_A8
